File: hardware/supplies.kicad_sch (KiCad schematic)
At the start: 20 parts, among them J11 Conn_01x02, J12 Conn_01x02, U8 AP62250WU

Commit message: HW: PCB Done
Parts:
- added D18: SMAJ14A, Diode_SMD:D_SMA, symbol Diode:SMAJ14A
- added H1, H2, H3, H4: MountingHole_Pad, MountingHole:MountingHole_3.2mm_M3_Pad, symbol Mechanical:MountingHole_Pad
- added NT4: NetTie_2, NetTie:NetTie-2_SMD_Pad2.0mm, symbol Device:NetTie_2
Connections:
- net GNDA: now also J12.2 (Pin_2), NT3.1, D18.2 (A2), H3.1, H4.1, NT4.1; no longer NT3.2
- net GNDPWR: now also NT3.2, H1.1, H2.1, NT4.2; no longer J12.2 (Pin_2), NT3.1
- net at J12.1 (Pin_1), JP16.2 (B): now also D18.1 (A1)
Other:
- moved on the sheet: NT3

Commit message: HW: Version 1.0
Parts:
- added J9: Barrel_Jack_MountingPin, Connector_BarrelJack:BarrelJack_GCT_DCJ200-10-A_Horizontal, symbol Connector:Barrel_Jack_MountingPin
- C19, C27, C28: footprint Capacitor_SMD:C_0805_2012Metric_Pad1.18x1.45mm_HandSolder -> Capacitor_SMD:C_0805_2012Metric
- C22, C23, C24: footprint Capacitor_SMD:C_1210_3225Metric_Pad1.33x2.70mm_HandSolder -> Capacitor_SMD:C_1210_3225Metric
- D11, D12: value Red Led 0805 -> YLED0805 Red; footprint LED_SMD:LED_0805_2012Metric_Pad1.15x1.40mm_HandSolder -> LED_SMD:LED_0805_2012Metric
- D18: LCSC Part (none) -> C99286
- L3: value 2.2uH 3A -> XFL4020-222MEC
- R40, R47, R52, R53, R54: footprint Resistor_SMD:R_0805_2012Metric_Pad1.20x1.40mm_HandSolder -> Resistor_SMD:R_0805_2012Metric
- U8: value AP62250WU -> AP62250WU-7; footprint Package_TO_SOT_SMD:TSOT-23-6_HandSoldering -> Package_TO_SOT_SMD:TSOT-23-6; LCSC Part (none) -> C5184228
Connections:
- net +12V: now also J12.1 (Pin_1)
- net GNDA: now also J9.2, J9.MP (MountPin)
- net at D18.1 (A1), JP16.2 (B): now also J9.1; no longer J12.1 (Pin_1)
- no-connect marks 0 -> 1
Other:
- moved on the sheet: D18, JP16
