File: hardware/supplies.kicad_sch (KiCad schematic)
At the start: 19 parts, among them J11 Conn_01x02, J12 Conn_01x02, U8 AP62250WU

Commit message: Hw/placa sepic (#34)
Co-authored-by: Federico Borello <156438142+fborello-lambda@users.noreply.github.com>
Parts:
- removed C22: 10uF 10% 50V X7R 0805, Capacitor_SMD:C_0805_2012Metric_Pad1.18x1.45mm_HandSolder, symbol Device:C_Polarized
- removed C26: 10uF 50V Aluminum Polymer, Capacitor_THT:CP_Radial_D6.3mm_P2.50mm, symbol Device:C_Polarized
- removed R39: 1K 1206, Resistor_SMD:R_0805_2012Metric_Pad1.20x1.40mm_HandSolder, symbol Device:R_US
- added C22, C23, C24: 22uF 10% 25V X7R 1210, Capacitor_SMD:C_1210_3225Metric, symbol Device:C
- added D18: SMAJ14A, Diode_SMD:D_SMA, symbol Diode:SMAJ14A
- added H1, H2, H3, H4: MountingHole_Pad, MountingHole:MountingHole_3.2mm_M3_Pad, symbol Mechanical:MountingHole_Pad
- added J9: Barrel_Jack_MountingPin, Connector_BarrelJack:BarrelJack_GCT_DCJ200-10-A_Horizontal, symbol Connector:Barrel_Jack_MountingPin
- added NT4: NetTie_2, NetTie:NetTie-2_SMD_Pad2.0mm, symbol Device:NetTie_2
- added R54: 4.7K 1% 0805, Resistor_SMD:R_0805_2012Metric, symbol Device:R_US
- C19, C27, C28: value 100nF 10% 100V X7R 0805 -> 100nF 10% 50V X7R 0805; footprint Capacitor_SMD:C_0805_2012Metric_Pad1.18x1.45mm_HandSolder -> Capacitor_SMD:C_0805_2012Metric
- D11, D12: value Red Led 0805 -> YLED0805 Red; footprint LED_SMD:LED_0805_2012Metric_Pad1.15x1.40mm_HandSolder -> LED_SMD:LED_0805_2012Metric; LCSC Part C19171391 -> (none)
- L3: value 4.7uH 3A -> XFL4020-222MEC; footprint (none) -> Inductor_SMD_Wurth:L_Wurth_WE-LQSH-4020; LCSC Part (none) -> C122469
- R40: value 150R -> 330R 1% 0805; footprint Resistor_SMD:R_0805_2012Metric_Pad1.20x1.40mm_HandSolder -> Resistor_SMD:R_0805_2012Metric; LCSC Part C153298 -> (none)
- R47: value 33K 0805 -> 33R 1% 0805; footprint Resistor_SMD:R_0805_2012Metric_Pad1.20x1.40mm_HandSolder -> Resistor_SMD:R_0805_2012Metric
- R52: value 10K 0805 -> 4.7K 1% 0805; footprint Resistor_SMD:R_0805_2012Metric_Pad1.20x1.40mm_HandSolder -> Resistor_SMD:R_0805_2012Metric; LCSC Part C153298 -> (none)
- R53: value 100K 0805 -> 100K 1% 0805; footprint Resistor_SMD:R_0805_2012Metric_Pad1.20x1.40mm_HandSolder -> Resistor_SMD:R_0805_2012Metric
- U8: value AP62250WU -> AP62250WU-7; LCSC Part (none) -> C5184228
Connections:
- net +12V: now also J12.1 (Pin_1), R54.1
- net +3.3V: now also C23.1, C24.1
- net GNDA: now also J12.2 (Pin_2), NT3.1, C22.2, C23.2, C24.2, D18.2 (A2), H3.1, H4.1, J9.2, J9.MP (MountPin), NT4.1; no longer NT3.2
- net GNDPWR: now also NT3.2, H1.1, H2.1, NT4.2; no longer J12.2 (Pin_2), NT3.1
- net at D11.2 (A): now also R54.2
- net at JP16.2 (B): now also D18.1 (A1), J9.1; no longer J12.1 (Pin_1)
- net at C19.1, JP17.2 (B), R53.1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: now also C22.1
- no-connect marks 0 -> 1
Other:
- moved on the sheet: C27, D11, D12, J11, JP16, NT3, R40
