File: hardware/untitled.kicad_sch (KiCad schematic)
At the start: 47 parts, among them J2 Conn_01x03 5.08mm, U1 MAX31865xTP, U2 INA229, U3 INA281A3

Commit message: HW: sch near final version
Parts:
- removed R3: 10mOhm 3W 1% 2512, Resistor_SMD:R_Shunt_Vishay_WSK2512_6332Metric_T1.19mm, symbol Device:R_Shunt_US
Connections:
- net Vin is gone; now on net VIN: U2.8 (VBUS)
- net VIN: no longer R4.1, R5.1, R6.1, R8.1, R9.1
- net VNEGA: no longer C1.2, C11.2, C12.2, C2.2, C4.2, C6.2, C7.2, C8.2, C9.2, D2.1 (A), D3.1 (A), R15.2, R7.2, U1.10 (GND), U1.15 (DGND), U1.16 (GND), U1.21 (GND), U2.7 (GND), U3.2 (GND)
- net ADC_Input_Current renamed ADC_Input_Curr
- net ADC_Input_Voltage renamed ADC_VPWR
- net ADC_Output_Voltage renamed ADC_VOUT
- net DRDY_TMP renamed DRDY_PT100
- net INA_OOR_ALERT renamed INA_OOR_Alert
- net SPIO0_CS1 renamed CS_INA
- net SPIO0_CS3 renamed CS_TP100
- net SPIO0_MISO renamed SPI_MISO
- net SPIO0_MOSI renamed SPI_MOSI
- net SPIO0_SCK renamed SPI_SCK
- net VPOSA renamed +3.3V
- new net GNDA: C1.2, C11.2, C12.2, C2.2, C4.2, C6.2, C7.2, C8.2, C9.2, D2.1 (A), D3.1 (A), R15.2, R7.2, U1.10 (GND), U1.15 (DGND), U1.16 (GND), U1.21 (GND), U2.7 (GND), U3.2 (GND)
- new net VPWR: R4.1, R5.1, R6.1, R8.1, R9.1

Commit message: HW: Sch done. PCB WIP
Parts:
- removed JP11, JP6: Jumper_2_Open, Connector_PinHeader_2.54mm:PinHeader_1x02_P2.54mm_Vertical, symbol Jumper:Jumper_2_Open
- removed R17, R9: R_US, Resistor_SMD:R_0805_2012Metric_Pad1.20x1.40mm_HandSolder, symbol Device:R_US
Connections:
- net VIN is gone; now on net VPWR: C6.1, U2.8 (VBUS)
