File: hardware/untitled.kicad_sch (KiCad schematic)
At the start: 42 parts, among them J2 Conn_01x03 5.08mm, U1 MAX31865xTP, U2 INA229, U3 INA281A3

Commit message: HW: PCB WIP
Parts:
- removed C1, C11, C7: 1uF 10% 50V X7R 0805, Capacitor_SMD:C_0805_2012Metric_Pad1.18x1.45mm_HandSolder, symbol Device:C_Polarized
- removed C12, C2, C8: 100nF 10% 100V X7R 0805, Capacitor_SMD:C_0805_2012Metric_Pad1.18x1.45mm_HandSolder, symbol Device:C
- removed JP2, JP3, JP4, JP5: Jumper_2_Open, Connector_PinHeader_2.54mm:PinHeader_1x02_P2.54mm_Vertical, symbol Jumper:Jumper_2_Open
- removed R4, R5, R6, R8: R_US, Resistor_SMD:R_0805_2012Metric_Pad1.20x1.40mm_HandSolder, symbol Device:R_US
- added C40, C42, C44: 1uF 10% 100V X7R 1206, Capacitor_SMD:C_1206_3216Metric_Pad1.33x1.80mm_HandSolder, symbol Device:C
- added C41, C43, C45: 100nF 10% 50V X7R 0805, Capacitor_SMD:C_0805_2012Metric_Pad1.18x1.45mm_HandSolder, symbol Device:C
- added JP11, JP13, JP14, JP6: Jumper_2_Open, Connector_PinHeader_2.54mm:PinHeader_1x02_P2.54mm_Vertical, symbol Jumper:Jumper_2_Open
- added R17, R30: 75K 1% 0805, Resistor_SMD:R_0805_2012Metric_Pad1.20x1.40mm_HandSolder, symbol Device:R_US
- C10, C3, C4, C5, C9: value 100nF 10% 100V X7R 0805 -> 100nF 10% 50V X7R 0805; LCSC Part C28233 -> (none)
- C6: value 1uF 10% 100V X7R 1210 -> 1uF 10% 100V X7R 1206; footprint Capacitor_SMD:C_1210_3225Metric_Pad1.33x2.70mm_HandSolder -> Capacitor_SMD:C_1206_3216Metric_Pad1.33x1.80mm_HandSolder; LCSC Part C382212 -> (none)
- JP1: LCSC Part C42431836 -> (none)
- JP10, JP7, JP8, JP9: LCSC Part C42431798 -> (none)
- R10, R11, R18, R19: value 10R 1% 0805 Resistor -> 10R 1% 0805; LCSC Part C2907220 -> (none)
- R12, R13, R14, R16: value R_US -> 75K 1% 0805
- R15, R7: value R_US -> 10K 1% 0805
- R2: value 400R 0.1% -> 400R 0.1% 0805; LCSC Part C153298 -> (none)
Connections:
- net +3.3V: now also C40.1, C41.1, C42.1, C43.1, C44.1, C45.1
- net ADC_VOUT: now also JP14.1 (A), R30.2; no longer JP10.1 (A), JP7.1 (A), JP8.1 (A), JP9.1 (A)
- net ADC_VPWR: now also R14.2, JP11.1 (A)
- net GNDA: now also C40.2, C41.2, C42.2, C43.2, C44.2, C45.2
- net VOUT: now also JP10.2 (B); no longer R12.1, R13.1, R14.1, R16.1
- net VPWR: now also JP9.2 (B); no longer C6.1, U2.8 (VBUS)
- net at R12.2: now also JP7.1 (A), R14.1, JP11.2 (B); no longer JP7.2 (B)
- net at R16.2: now also JP8.1 (A), JP13.2 (B), R17.1; no longer JP10.2 (B)
- net at R13.2: now also JP7.2 (B), R12.1, JP6.1 (A); no longer JP8.2 (B)
- new net: JP10.1 (A), JP8.2 (B), R16.1
- new net: JP13.1 (A), JP14.2 (B), R17.2, R30.1
- new net: JP6.2 (B), JP9.1 (A), R13.1
- new net VIN: C6.1, U2.8 (VBUS)
Other:
- moved on the sheet: C4, C5, C6, C9, D2, D3, R10, R11, R15, R18, R19, R7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

Commit message: HW: PCB Done
Parts:
- removed JP11, JP14: Jumper_2_Open, Connector_PinHeader_2.54mm:PinHeader_1x02_P2.54mm_Vertical, symbol Jumper:Jumper_2_Open
