File: hardware/Pico.kicad_sch (KiCad schematic)
At the start: 14 parts, among them J1 Conn_01x03 2.54mm, J5 Conn_01x04, J6 Conn_01x06, J7 Conn_01x12

Commit message: HW: Sch done. PCB WIP
Parts:
- removed JP12: Jumper_2_Open, symbol Jumper:Jumper_2_Open
- added C25: 3.3nF 10% 100V X7R 0805, Capacitor_SMD:C_0805_2012Metric_Pad1.18x1.45mm_HandSolder, symbol Device:C
- added D10, D13: BAT54S, Package_TO_SOT_SMD:SOT-23, symbol Diode:BAT54S
- added JP12: 2/3 Wire Selector, Connector_PinHeader_2.54mm:PinHeader_1x03_P2.54mm_Vertical, symbol Jumper:Jumper_3_Open
- added R32: 10R 1%, Resistor_SMD:R_0805_2012Metric_Pad1.20x1.40mm_HandSolder, symbol Device:R_US
- added R33, R34, R35, R36, R41, R42, R43, R44, R45, R46: 330R 1%, Resistor_SMD:R_0805_2012Metric_Pad1.20x1.40mm_HandSolder, symbol Device:R_US
- added R48, R49, R50, R51: 33R 1%, Resistor_SMD:R_0805_2012Metric_Pad1.20x1.40mm_HandSolder, symbol Device:R_US
- added U10, U6, U7, U9: SRV05-4, Package_TO_SOT_SMD:SOT-23-6, symbol Power_Protection:SRV05-4
- J5: footprint (none) -> Connector_PinHeader_2.54mm:PinHeader_1x04_P2.54mm_Vertical; now left out of the parts list
- J6: footprint (none) -> Connector_PinHeader_2.54mm:PinHeader_1x06_P2.54mm_Vertical; now left out of the parts list
- J7: footprint (none) -> Connector_PinHeader_2.54mm:PinHeader_1x12_P2.54mm_Vertical; now left out of the parts list
Connections:
- net +3.3V: now also R21.2, R22.2, JP12.2 (C), U10.5 (VP), U6.5 (VP), U7.5 (VP), U9.5 (VP)
- net Blinky: now also R45.1; no longer J7.11 (Pin_11)
- net GNDA: now also C25.2, U10.2 (VN), U6.2 (VN), U7.2 (VN), U9.2 (VN); no longer R21.2, R22.2
- net GPIO1: now also R35.1; no longer J7.5 (Pin_5)
- net GPIO2: now also R36.1; no longer J7.6 (Pin_6)
- net GPIO3: now also R41.1; no longer J7.7 (Pin_7)
- net GPIO4: now also R42.1; no longer J7.8 (Pin_8)
- net GPIO5: now also R43.1; no longer J7.9 (Pin_9)
- net GPIO6: now also R44.1; no longer J7.10 (Pin_10)
- net I2C_SCL: now also U9.6 (IO4)
- net I2C_SDA: now also U9.4 (IO3)
- net LED1: now also R33.1; no longer J7.3 (Pin_3)
- net LED2: now also R34.1; no longer J7.4 (Pin_4)
- net PWM_Gate: now also C25.1, R32.1, R46.1; no longer A1.20 (GPIO15), J7.12 (Pin_12)
- net SPI1_CS: now also R51.1; no longer J6.5 (Pin_5)
- net SPI1_RX: now also R50.1; no longer J6.4 (Pin_4)
- net SPI1_SCK: now also R48.1; no longer J6.2 (Pin_2)
- net SPI1_TX: now also R49.1; no longer J6.3 (Pin_3)
- net at A1.36 (3V3): now also D13.1 (A)
- net at A1.39 (VSYS): now also D10.2 (K)
- new net: D13.3 (COM), JP12.1 (A)
- new net: D10.3 (COM), JP12.3 (B)
- new net: A1.20 (GPIO15), R32.2
- new net OUT_CS: J6.5 (Pin_5), R51.2, U10.6 (IO4)
- new net OUT_RX: J6.4 (Pin_4), R50.2, U10.4 (IO3)
- new net OUT_SCK: J6.2 (Pin_2), R48.2, U10.1 (IO1)
- new net OUT_TX: J6.3 (Pin_3), R49.2, U10.3 (IO2)
- new net Out1: J7.3 (Pin_3), R33.2, U6.1 (IO1)
- new net Out10: J7.12 (Pin_12), R46.2, U9.3 (IO2)
- new net Out2: J7.4 (Pin_4), R34.2, U6.3 (IO2)
- new net Out3: J7.5 (Pin_5), R35.2, U6.4 (IO3)
- new net Out4: J7.6 (Pin_6), R36.2, U6.6 (IO4)
- new net Out5: J7.7 (Pin_7), R41.2, U7.1 (IO1)
- new net Out6: J7.8 (Pin_8), R42.2, U7.3 (IO2)
- new net Out7: J7.9 (Pin_9), R43.2, U7.4 (IO3)
- new net Out8: J7.10 (Pin_10), R44.2, U7.6 (IO4)
- new net Out9: J7.11 (Pin_11), R45.2, U9.1 (IO1)
Other:
- note removed: "SPIO: SPI Channel for Sensors. SPI1: SPI Channel for Duty/Reference Input. CS1: Input V/I INA CS2: CS3: PT100 Sensor"
- moved on the sheet: A1, D6, D7, D8, J1, J5, J6, J7, R21, R22, R24, R26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

Commit message: HW: Changes in GPIO components. PCB WIP
Parts:
- removed D7, D8: Red Led 0805, LED_SMD:LED_0805_2012Metric_Pad1.15x1.40mm_HandSolder, symbol Device:LED
- removed R31: 150R, Resistor_SMD:R_0805_2012Metric_Pad1.20x1.40mm_HandSolder, symbol Device:R_US
- added C13, C18, C20, C21: 100nF 10% 100V X7R 0805, Capacitor_SMD:C_0805_2012Metric_Pad1.18x1.45mm_HandSolder, symbol Device:C
- added D14, D15, D7, D8: WS2812, LED_SMD:LED_WS2812_PLCC6_5.0x5.0mm_P1.6mm, symbol LED:WS2812
- added J8: Conn_01x04, Connector_PinHeader_2.54mm:PinHeader_1x04_P2.54mm_Vertical, symbol Connector_Generic:Conn_01x04
- added R28: 4.7K, Resistor_SMD:R_0805_2012Metric_Pad1.20x1.40mm_HandSolder, symbol Device:R_US
- added SW1, SW2: SW_SPST, Button_Switch_SMD:SW_Push_1TS009xxxx-xxxx-xxxx_6x6x5mm, symbol Switch:SW_SPST
- R26: value 150R -> 4.7K; LCSC Part C153298 -> (none)
Connections:
- net LED2 is gone; now on net But2: A1.2 (GPIO1), R34.1
- net +3.3V: now also R26.1, C13.1, C18.1, C20.1, C21.1, D14.3 (VCC), D14.5 (VDD), D15.3 (VCC), D15.5 (VDD), D7.3 (VCC), D7.5 (VDD), D8.3 (VCC), D8.5 (VDD), J8.1 (Pin_1), R28.1
- net GNDA: now also C13.2, C18.2, C20.2, C21.2, D14.6 (VSS), D15.6 (VSS), D7.6 (VSS), D8.6 (VSS), J8.2 (Pin_2), SW1.2 (B), SW2.2 (B)
- net GPIO1: now also D7.2 (DIN)
- net I2C_SCL: now also J8.4 (Pin_4)
- net I2C_SDA: now also J8.3 (Pin_3)
- net But2: now reaches R26.2
- net But2: now also SW1.1 (A)
- net LED1 renamed But1
- net But1: now also R28.2, SW2.1 (A); no longer R26.1
- new net: D14.1 (DOUT), D15.2 (DIN)
- new net: D7.1 (DOUT), D8.2 (DIN)
- new net: D14.2 (DIN), D8.1 (DOUT)
- no-connect marks 0 -> 1
Other:
- moved on the sheet: A1, C25, D10, D13, D6, J1, J5, J6, J7, JP12, R21, R22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

Commit message: HW: PCB WIP
Parts:
- C13, C18, C20, C21: value 100nF 10% 100V X7R 0805 -> 100nF 10% 50V X7R 0805; LCSC Part C28233 -> (none)
- C25: value 3.3nF 10% 100V X7R 0805 -> 1nF 1KV X7R 1206; footprint Capacitor_SMD:C_0805_2012Metric_Pad1.18x1.45mm_HandSolder -> Capacitor_SMD:C_1206_3216Metric_Pad1.33x1.80mm_HandSolder
- D6: LCSC Part C19171391 -> (none)
- JP12: LCSC Part C42431836 -> (none)
- R21, R22: value 4.7Kohm -> 4.7K 1% 0805; LCSC Part C153298 -> (none)
- R24: value 150R -> 330R 1% 0805; LCSC Part C153298 -> (none)
- R26, R28: value 4.7K -> 4.7K 1% 0805
- R32: value 10R 1% -> 33R 1% 0805
- R33, R34, R35, R36, R41, R42, R43, R44, R45, R46: value 330R 1% -> 330R 1% 0805
- R48, R49, R50, R51: value 33R 1% -> 33R 1% 0805
Connections:
- net GPIO3 is gone; now on net GPIO4: A1.6 (GPIO4), R41.1
- net GPIO4: now also D7.2 (DIN); no longer A1.10 (GPIO7), R42.1
- net I2C_SCL: now also U9.1 (IO1); no longer U9.6 (IO4)
- net I2C_SDA: now also U9.3 (IO2); no longer U9.4 (IO3)
- net OUT_CS: now also U10.4 (IO3); no longer U10.6 (IO4)
- net OUT_RX: now also U10.6 (IO4); no longer U10.4 (IO3)
- net OUT_SCK: now also U10.3 (IO2); no longer U10.1 (IO1)
- net OUT_TX: now also U10.1 (IO1); no longer U10.3 (IO2)
- net Out1: now also U6.3 (IO2); no longer U6.1 (IO1)
- net Out10: now also U9.4 (IO3); no longer U9.3 (IO2)
- net Out2: now also U6.1 (IO1); no longer U6.3 (IO2)
- net Out3: now also U6.6 (IO4); no longer U6.4 (IO3)
- net Out4: now also U6.4 (IO3); no longer U6.6 (IO4)
- net Out5: now also U7.3 (IO2); no longer U7.1 (IO1)
- net Out6: now also U7.1 (IO1); no longer U7.3 (IO2)
- net Out7: now also U7.6 (IO4); no longer U7.4 (IO3)
- net Out8: now also U7.4 (IO3); no longer U7.6 (IO4)
- net Out9: now also U9.6 (IO4); no longer U9.1 (IO1)
- net GPIO1 renamed Tracer_En
- net Tracer_En: no longer D7.2 (DIN)
- net GPIO2 renamed Tracer_pwm
- net GPIO5 renamed GPIO8
- net GPIO6 renamed GPIO9
- new net GPIO7: A1.10 (GPIO7), R42.1
- no-connect marks 1 -> 7
Other:
- moved on the sheet: A1, C13, C18, C20, C21, C25, D10, D13, D14, D15, D7, D8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

Commit message: HW: Version 1.0
Parts:
- removed D14, D15, D7, D8: WS2812, LED_SMD:LED_WS2812_PLCC6_5.0x5.0mm_P1.6mm, symbol LED:WS2812
- added D19, D20, D21, D22: WS2812B, LED_SMD:LED_WS2812B_PLCC4_5.0x5.0mm_P3.2mm, symbol LED:WS2812B
- C13, C18, C20, C21: footprint Capacitor_SMD:C_0805_2012Metric_Pad1.18x1.45mm_HandSolder -> Capacitor_SMD:C_0805_2012Metric
- C25: value 1nF 1KV X7R 1206 -> 1nF 10% 1KV X7R 1206; footprint Capacitor_SMD:C_1206_3216Metric_Pad1.33x1.80mm_HandSolder -> Capacitor_SMD:C_1206_3216Metric
- D10, D13: value BAT54S -> BAT54SLT1G
- D6: value Red Led 0805 -> YLED0805 Red; footprint LED_SMD:LED_0805_2012Metric_Pad1.15x1.40mm_HandSolder -> LED_SMD:LED_0805_2012Metric
- J1: LCSC Part C42431836 -> (none)
- R21, R22, R24, R26, R28, R32, R33, R34, R35, R36, R41, R42, R43, R44, R45, R46, R48, R49, R50, R51: footprint Resistor_SMD:R_0805_2012Metric_Pad1.20x1.40mm_HandSolder -> Resistor_SMD:R_0805_2012Metric
- SW1, SW2: value SW_SPST -> 1TS009A-1800-5000-CT; LCSC Part (none) -> C319409
- U10, U6, U7, U9: LCSC Part (none) -> C1975211
Connections:
- net +3.3V: now also D19.1 (VDD), D20.1 (VDD), D21.1 (VDD), D22.1 (VDD)
- net GNDA: now also D19.3 (VSS), D20.3 (VSS), D21.3 (VSS), D22.3 (VSS)
- net GPIO4: now also D19.4 (DIN)
- new net: D20.2 (DOUT), D21.4 (DIN)
- new net: D19.2 (DOUT), D20.4 (DIN)
- new net: D21.2 (DOUT), D22.4 (DIN)
