File: hardware/Proyecto0.1V.kicad_pcb (KiCad board)
At the start: 2 copper layers, 121 parts, among them J1 Conn_01x03 2.54mm, J11 Conn_01x02, J12 Conn_01x02, J13 Conn_01x02, J14 Conn_01x02, J2 Conn_01x03 5.08mm, J3 Conn_01x04 5.08mm, J4 Conn_01x04 5.08mm, J5 Conn_01x04, J6 Conn_01x06, J7 Conn_01x12, Q2 IPP200N25N3, U1 MAX31865xTP, U10 SRV05-4, U2 INA229, U3 INA281A3, U4 TC4422, U6 SRV05-4, U7 SRV05-4, U8 AP62250WU, U9 SRV05-4

Commit message: HW: Changes in GPIO components. PCB WIP
Parts:
- moved Q2 158.7 mm to (205.6, 53.8), turned to 0 degrees
- moved R27 151.3 mm to (205.6, 61.5), turned to 180 degrees
- moved L1 143.5 mm to (185.7, 83.8), turned to 90 degrees
- moved C16 143.5 mm to (213.2, 61.5), turned to 180 degrees
- moved C14 131.8 mm to (205.6, 86.9), turned to 0 degrees
- moved J13 128.4 mm to (144.8, 102.9), turned to 180 degrees
- moved D5 121.7 mm to (152.4, 100.4), turned to 0 degrees
- moved D9 121.6 mm to (147.4, 108.0), turned to 90 degrees
- moved C17 118.4 mm to (236.0, 68.6)
- moved R23 117.5 mm to (152.4, 105.5), turned to 180 degrees
- moved D4 116.1 mm to (192.9, 106.1)
- moved R20 115.5 mm to (152.4, 108.0), turned to 180 degrees
- moved J2 114.4 mm to (50.8, 111.8), turned to -90 degrees
- moved A1 111.8 mm to (87.6, 80.0)
- moved J1 111.8 mm to (85.1, 115.6)
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
Commit message: HW: PCB WIP
Parts:
- removed C1, C11, C7: 1uF 10% 50V X7R 0805, Capacitor_SMD:C_0805_2012Metric_Pad1.18x1.45mm_HandSolder
- removed C12, C2, C8: 100nF 10% 100V X7R 0805, Capacitor_SMD:C_0805_2012Metric_Pad1.18x1.45mm_HandSolder
- removed C26: 10uF 50V Aluminum Polymer, Capacitor_THT:CP_Radial_D6.3mm_P2.50mm
- removed JP2, JP3, JP4, JP5: Jumper_2_Open, Connector_PinHeader_2.54mm:PinHeader_1x02_P2.54mm_Vertical
- removed R39: 1K 1206, Resistor_SMD:R_0805_2012Metric_Pad1.20x1.40mm_HandSolder
- added C13: 100nF 10% 50V X7R 0805, Capacitor_SMD:C_0805_2012Metric_Pad1.18x1.45mm_HandSolder, F.Cu at (110.7, 66.5)
- added C18: 100nF 10% 50V X7R 0805, Capacitor_SMD:C_0805_2012Metric_Pad1.18x1.45mm_HandSolder, F.Cu at (110.7, 79.2)
- added C20: 100nF 10% 50V X7R 0805, Capacitor_SMD:C_0805_2012Metric_Pad1.18x1.45mm_HandSolder, F.Cu at (120.9, 66.5)
- added C21: 100nF 10% 50V X7R 0805, Capacitor_SMD:C_0805_2012Metric_Pad1.18x1.45mm_HandSolder, F.Cu at (120.9, 79.2)
- added C29: C, Capacitor_SMD:C_0805_2012Metric_Pad1.18x1.45mm_HandSolder, F.Cu at (101.6, 124.5)
- added C30: C, Capacitor_SMD:C_0805_2012Metric_Pad1.18x1.45mm_HandSolder, F.Cu at (106.7, 127.0)
- added C31: C, Capacitor_SMD:C_0805_2012Metric_Pad1.18x1.45mm_HandSolder, F.Cu at (106.7, 116.8)
- added C33: 100nF 10% 50V X7R 0805, Capacitor_SMD:C_0805_2012Metric_Pad1.18x1.45mm_HandSolder, F.Cu at (111.8, 119.4)
- added C34: 100nF 10% 50V X7R 0805, Capacitor_SMD:C_0805_2012Metric_Pad1.18x1.45mm_HandSolder, F.Cu at (125.1, 99.1)
- added C37: 1uF 10% 100V X7R 1206, Capacitor_SMD:C_1206_3216Metric_Pad1.33x1.80mm_HandSolder, F.Cu at (111.8, 116.8)
- added C38: 1uF 10% 100V X7R 1206, Capacitor_SMD:C_1206_3216Metric_Pad1.33x1.80mm_HandSolder, F.Cu at (125.1, 102.9)
- added C40: 1uF 10% 100V X7R 1206, Capacitor_SMD:C_1206_3216Metric_Pad1.33x1.80mm_HandSolder, F.Cu at (59.7, 115.6)
- added C41: 100nF 10% 50V X7R 0805, Capacitor_SMD:C_0805_2012Metric_Pad1.18x1.45mm_HandSolder, F.Cu at (53.3, 116.8)
- added C42: 1uF 10% 100V X7R 1206, Capacitor_SMD:C_1206_3216Metric_Pad1.33x1.80mm_HandSolder, F.Cu at (88.9, 124.5)
- added C43: 100nF 10% 50V X7R 0805, Capacitor_SMD:C_0805_2012Metric_Pad1.18x1.45mm_HandSolder, F.Cu at (82.5, 124.5)
- added C44: 1uF 10% 100V X7R 1206, Capacitor_SMD:C_1206_3216Metric_Pad1.33x1.80mm_HandSolder, F.Cu at (71.1, 125.7)
- added C45: 100nF 10% 50V X7R 0805, Capacitor_SMD:C_0805_2012Metric_Pad1.18x1.45mm_HandSolder, F.Cu at (76.2, 124.5)
- added D14: WS2812, LED_SMD:LED_WS2812_PLCC6_5.0x5.0mm_P1.6mm, F.Cu at (120.9, 84.3)
- added D15: WS2812, LED_SMD:LED_WS2812_PLCC6_5.0x5.0mm_P1.6mm, F.Cu at (120.9, 71.6)
- added D16: MBRB20200, Package_TO_SOT_SMD:TO-263-2, F.Cu at (250.2, 33.7)
- added D17: SS110, Diode_SMD:D_SMA_Handsoldering, F.Cu at (150.9, 126.1)
- added J8: Conn_01x04, Connector_PinHeader_2.54mm:PinHeader_1x04_P2.54mm_Vertical, F.Cu at (53.3, 73.7)
- added JP11: Jumper_2_Open, Connector_PinHeader_2.54mm:PinHeader_1x02_P2.54mm_Vertical, F.Cu at (138.4, 101.6)
- added JP13: Jumper_2_Open, Connector_PinHeader_2.54mm:PinHeader_1x02_P2.54mm_Vertical, F.Cu at (142.2, 78.7)
- added JP14: Jumper_2_Open, Connector_PinHeader_2.54mm:PinHeader_1x02_P2.54mm_Vertical, F.Cu at (138.4, 78.7)
- added JP6: Jumper_2_Open, Connector_PinHeader_2.54mm:PinHeader_1x02_P2.54mm_Vertical, F.Cu at (146.1, 101.6)
- added K1: G5LE-1, Relay_THT:Relay_SPDT_Omron-G5LE-1, F.Cu at (158.5, 126.1)
- added Q1: MMBT3904, Package_TO_SOT_SMD:SOT-23, F.Cu at (143.3, 126.1)
- added Q3: IPP200N25N3, Package_TO_SOT_THT:TO-220-3_Vertical, F.Cu at (138.2, 113.4)
- added R1: R_US, Resistor_SMD:R_0805_2012Metric_Pad1.20x1.40mm_HandSolder, F.Cu at (101.6, 121.9)
- added R17: 75K 1% 0805, Resistor_SMD:R_0805_2012Metric_Pad1.20x1.40mm_HandSolder, F.Cu at (149.9, 86.4)
- added R28: 4.7K 1% 0805, Resistor_SMD:R_0805_2012Metric_Pad1.20x1.40mm_HandSolder, F.Cu at (66.0, 53.3)
- added R29: 10m 3W 1% 2512, Resistor_SMD:R_2512_6332Metric_Pad1.40x3.35mm_HandSolder, F.Cu at (150.9, 113.4)
- added R3: R_US, Resistor_SMD:R_0805_2012Metric_Pad1.20x1.40mm_HandSolder, F.Cu at (101.6, 127.0)
- added R30: 75K 1% 0805, Resistor_SMD:R_0805_2012Metric_Pad1.20x1.40mm_HandSolder, F.Cu at (147.3, 86.4)
- added R37: 4.7K 1% 0805, Resistor_SMD:R_0805_2012Metric_Pad1.20x1.40mm_HandSolder, F.Cu at (140.7, 131.2)
- added R54: 4.7K 1% 0805, Resistor_SMD:R_0805_2012Metric_Pad1.20x1.40mm_HandSolder, F.Cu at (132.1, 56.5)
- added SW1: SW_SPST, Button_Switch_SMD:SW_Push_1TS009xxxx-xxxx-xxxx_6x6x5mm, F.Cu at (41.9, 63.5)
- added SW2: SW_SPST, Button_Switch_SMD:SW_Push_1TS009xxxx-xxxx-xxxx_6x6x5mm, F.Cu at (41.9, 53.3)
- added U5: MCP601-xOT, Package_TO_SOT_SMD:SOT-23-5, F.Cu at (106.7, 121.9)
- C10, C19, C27, C28, C3, C4, C5, C9: value 100nF 10% 100V X7R 0805 -> 100nF 10% 50V X7R 0805
- C16: value 1nF 1000V -> 1nF 1KV X7R 1206; footprint Capacitor_SMD:C_1210_3225Metric_Pad1.33x2.70mm_HandSolder -> Capacitor_SMD:C_1206_3216Metric_Pad1.33x1.80mm_HandSolder
- C22: value 10uF 10% 50V X7R 0805 -> 22uF 10% 25V X7R 1210; footprint Capacitor_SMD:C_0805_2012Metric_Pad1.18x1.45mm_HandSolder -> Capacitor_SMD:C_1210_3225Metric_Pad1.33x2.70mm_HandSolder
- C23: value 1uF 10% 50V X7R 0805 -> 22uF 10% 25V X7R 1210; footprint Capacitor_SMD:C_0805_2012Metric_Pad1.18x1.45mm_HandSolder -> Capacitor_SMD:C_1210_3225Metric_Pad1.33x2.70mm_HandSolder
- C24: value 10uF 50V Aluminum Polymer -> 22uF 10% 25V X7R 1210; footprint Capacitor_THT:CP_Radial_D6.3mm_P2.50mm -> Capacitor_SMD:C_1210_3225Metric_Pad1.33x2.70mm_HandSolder
- C25: value 3.3nF 10% 100V X7R 0805 -> 1nF 1KV X7R 1206; footprint Capacitor_SMD:C_0805_2012Metric_Pad1.18x1.45mm_HandSolder -> Capacitor_SMD:C_1206_3216Metric_Pad1.33x1.80mm_HandSolder
- C6: value 1uF 10% 100V X7R 1210 -> 1uF 10% 100V X7R 1206; footprint Capacitor_SMD:C_1210_3225Metric_Pad1.33x2.70mm_HandSolder -> Capacitor_SMD:C_1206_3216Metric_Pad1.33x1.80mm_HandSolder
- D1, D5: footprint Diode_SMD:D_SMA -> Diode_SMD:D_SMA_Handsoldering
- D7, D8: value Red Led 0805 -> WS2812; footprint LED_SMD:LED_0805_2012Metric_Pad1.15x1.40mm_HandSolder -> LED_SMD:LED_WS2812_PLCC6_5.0x5.0mm_P1.6mm
- L3: value 4.7uH 3A -> 2.2uH 3A; footprint Inductor_SMD:L_12x12mm_H8mm -> Inductor_SMD_Wurth:L_Wurth_WE-LQSH-4020
- R10, R11, R18, R19: value 10R 1% 0805 Resistor -> 10R 1% 0805
- R12, R13, R14, R16: value R_US -> 75K 1% 0805
- R15, R7: value R_US -> 10K 1% 0805
- R2: value 400R 0.1% -> 400R 0.1% 0805
- R20: value 33R 1% 0805 Resistor -> 33R 1% 0805
- R21, R22: value 4.7Kohm -> 4.7K 1% 0805
- R23: value 10K 1% 0805 Resistor -> 10K 1% 0805
- R24, R40: value 150R -> 330R 1% 0805
- R25: value 10mOhm 3W 1% 2512 -> 10m 3W 1% 2512
- R26, R31: value 150R -> 4.7K 1% 0805
- R27: value 4.7R Ohm 3W 1% 2512 -> 4.7R 3W 1% 2512
- R32: value 10R 1% -> 33R 1% 0805
- R33, R34, R35, R36, R41, R42, R43, R44, R45, R46: value 330R 1% -> 330R 1% 0805
- R47: value 33K 0805 -> 33R 1% 0805
- R48, R49, R50, R51: value 33R 1% -> 33R 1% 0805
- R52: value 10K 0805 -> 4.7K 1% 0805
- R53: value 100K 0805 -> 100K 1% 0805
- U8: footprint Package_TO_SOT_SMD:TSOT-23-6 -> Package_TO_SOT_SMD:TSOT-23-6_HandSoldering
- moved R31 105.2 mm to (143.3, 131.2), turned to -90 degrees
- moved R4 78.4 mm to (111.8, 127.0)
- moved J13 71.9 mm to (195.6, 52.1), turned to -90 degrees
- moved R5 70.6 mm to (101.6, 119.4), turned to 0 degrees
- moved R6 64.0 mm to (101.6, 116.8), turned to 0 degrees
- moved C24 60.8 mm to (142.9, 56.5), turned to -90 degrees
- moved R8 59.3 mm to (111.8, 121.9)
- moved C23 57.1 mm to (146.7, 56.5), turned to -90 degrees
- moved C5 57.0 mm to (76.2, 119.4), turned to 180 degrees
- moved R11 56.3 mm to (76.2, 121.9), turned to 180 degrees
- moved U2 56.1 mm to (68.6, 120.7)
- moved R10 55.8 mm to (76.2, 116.8), turned to 180 degrees
- moved D7 53.4 mm to (110.7, 84.3), turned to 90 degrees
- moved C6 52.4 mm to (71.1, 115.6), turned to 180 degrees
- moved D1 46.1 mm to (110.5, 94.0), turned to 0 degrees
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Connections:
- net /Pico/GPIO2 renamed /Pico/Tracer_pwm
- net /Pico/GPIO5 renamed /Pico/GPIO8
- net /Pico/GPIO6 renamed /Pico/GPIO9
- A1 pad 1: /Pico/LED1 -> /Pico/But1
- A1 pad 10: /Pico/GPIO4 -> /Pico/GPIO7
- A1 pad 2: /Pico/LED2 -> /Pico/But2
- A1 pad 4: /Pico/GPIO1 -> /Pico/Tracer_En
- A1 pad 6: /Pico/GPIO3 -> /Pico/GPIO4
- C23 pad 1: +12V -> +3.3V
- C23 pad 2: GNDPWR -> GNDA
- C24 pad 1: +12V -> +3.3V
- C24 pad 2: GNDPWR -> GNDA
- C6 pad 1: /AnalogConverters/VPWR -> /AnalogConverters/VIN
- D7 pad 1: GNDA -> Net-(D7-DOUT)
- D7 pad 2: Net-(D7-A) -> /Pico/GPIO4
- D8 pad 1: GNDA -> Net-(D14-DIN)
- D8 pad 2: Net-(D8-A) -> Net-(D7-DOUT)
- J3 pad 1: /SepicConverter/VIN -> /AnalogConverters/VIN
- J3 pad 2: /SepicConverter/VIN -> /AnalogConverters/VIN
- JP10 pad 1: /AnalogConverters/ADC_VOUT -> Net-(JP10-A)
- JP10 pad 2: Net-(JP10-B) -> /AnalogConverters/VOUT
- JP7 pad 1: /AnalogConverters/ADC_VOUT -> Net-(JP11-B)
- JP7 pad 2: Net-(JP7-B) -> Net-(JP6-A)
- JP8 pad 1: /AnalogConverters/ADC_VOUT -> Net-(JP13-B)
- JP8 pad 2: Net-(JP8-B) -> Net-(JP10-A)
- JP9 pad 1: /AnalogConverters/ADC_VOUT -> Net-(JP6-B)
- JP9 pad 2: Net-(JP9-B) -> /AnalogConverters/VPWR
- NT1 pad 1: /SepicConverter/VIN -> /AnalogConverters/VIN
- NT2 pad 1: /AnalogConverters/VPWR -> Net-(K1-Pad1)
- R12 pad 1: /AnalogConverters/VOUT -> Net-(JP6-A)
- R12 pad 2: Net-(JP7-B) -> Net-(JP11-B)
- R13 pad 1: /AnalogConverters/VOUT -> Net-(JP6-B)
- R13 pad 2: Net-(JP8-B) -> Net-(JP6-A)
- R14 pad 1: /AnalogConverters/VOUT -> Net-(JP11-B)
- R14 pad 2: Net-(JP9-B) -> /AnalogConverters/ADC_VPWR
- R16 pad 1: /AnalogConverters/VOUT -> Net-(JP10-A)
- R16 pad 2: Net-(JP10-B) -> Net-(JP13-B)
- R25 pad 1: /SepicConverter/VIN -> /AnalogConverters/VIN
- R25 pad 2: /AnalogConverters/VPWR -> Net-(K1-Pad1)
- R26 pad 1: /Pico/LED1 -> +3.3V
- R26 pad 2: Net-(D7-A) -> /Pico/But2
- R31 pad 1: /Pico/LED2 -> Net-(Q1-B)
- R31 pad 2: Net-(D8-A) -> /Pico/Tracer_En
- R33 pad 1: /Pico/LED1 -> /Pico/But1
- R34 pad 1: /Pico/LED2 -> /Pico/But2
- R35 pad 1: /Pico/GPIO1 -> /Pico/Tracer_En
- R4 pad 1: /AnalogConverters/VPWR -> GNDA
- R41 pad 1: /Pico/GPIO3 -> /Pico/GPIO4
- R42 pad 1: /Pico/GPIO4 -> /Pico/GPIO7
- R5 pad 1: /AnalogConverters/VPWR -> GNDA
- R5 pad 2: Net-(JP3-B) -> Net-(C31-Pad1)
- R6 pad 1: /AnalogConverters/VPWR -> Net-(Q3-G)
- R6 pad 2: Net-(JP4-B) -> Net-(C31-Pad1)
- R8 pad 1: /AnalogConverters/VPWR -> Net-(Q3-S)
- U10 pad 1: /Pico/OUT_SCK -> /Pico/OUT_TX
- U10 pad 3: /Pico/OUT_TX -> /Pico/OUT_SCK
- U10 pad 4: /Pico/OUT_RX -> /Pico/OUT_CS
- U10 pad 6: /Pico/OUT_CS -> /Pico/OUT_RX
- U2 pad 8: /AnalogConverters/VPWR -> /AnalogConverters/VIN
- U6 pad 1: /Pico/Out1 -> /Pico/Out2
- U6 pad 3: /Pico/Out2 -> /Pico/Out1
- U6 pad 4: /Pico/Out3 -> /Pico/Out4
- U6 pad 6: /Pico/Out4 -> /Pico/Out3
- U7 pad 1: /Pico/Out5 -> /Pico/Out6
- U7 pad 3: /Pico/Out6 -> /Pico/Out5
- U7 pad 4: /Pico/Out7 -> /Pico/Out8
- U7 pad 6: /Pico/Out8 -> /Pico/Out7
- U9 pad 1: /Pico/Out9 -> /Pico/I2C_SCL
- U9 pad 3: /Pico/Out10 -> /Pico/I2C_SDA
- U9 pad 4: /Pico/I2C_SDA -> /Pico/Out10
- U9 pad 6: /Pico/I2C_SCL -> /Pico/Out9
Routing:
- net GNDA: track 0.00 -> 129.9 mm, vias 0 -> 54
- net +3.3V: track 0.00 -> 95.8 mm, vias 0 -> 28
- net Net-(D14-DIN): track 0.00 -> 51.7 mm
- net /Pico/Out4: track 0.00 -> 51.2 mm
- net /Pico/But2: track 0.00 -> 50.4 mm, vias 0 -> 2
- net /Pico/I2C_SDA: track 0.00 -> 50.2 mm, vias 0 -> 2
- net /Pico/Out2: track 0.00 -> 49.6 mm, vias 0 -> 2
- net /Pico/Out3: track 0.00 -> 49.1 mm, vias 0 -> 2
- net /Pico/Out1: track 0.00 -> 48.3 mm
- net /Pico/I2C_SCL: track 0.00 -> 48.3 mm, vias 0 -> 2
- net /Pico/But1: track 0.00 -> 37.8 mm
- net /Pico/PWM_Gate: track 0.00 -> 37.1 mm, vias 0 -> 2
- net /Pico/Blinky: track 0.00 -> 30.4 mm, vias 0 -> 2
- net Net-(J2-Pin_2): track 0.00 -> 29.1 mm, vias 0 -> 1
- net Net-(J2-Pin_1): track 0.00 -> 25.3 mm
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Other:
- board text added: "C4"
- board text added: "JP6"
- board text added: "JP7"
- board text added: "JP9"
- board text added: "R7"

Commit message: HW: PCB Done
Parts:
- removed JP11, JP14: Jumper_2_Open, Connector_PinHeader_2.54mm:PinHeader_1x02_P2.54mm_Vertical
- added D18: SMAJ14A, Diode_SMD:D_SMA, F.Cu at (139.5, 63.0)
- added G***: LOGO, Custom_Library:logo_Grupo, F.Cu at (195.6, 56.1)
- added G***: LOGO, Custom_Library:UTN_LOGO, F.Cu at (197.9, 124.5)
- added H1: MountingHole_Pad, MountingHole:MountingHole_3.2mm_M3_Pad, F.Cu at (204.7, 56.0)
- added H2: MountingHole_Pad, MountingHole:MountingHole_3.2mm_M3_Pad, F.Cu at (204.7, 122.0)
- added H3: MountingHole_Pad, MountingHole:MountingHole_3.2mm_M3_Pad, F.Cu at (39.0, 123.0)
- added H4: MountingHole_Pad, MountingHole:MountingHole_3.2mm_M3_Pad, F.Cu at (39.0, 57.0)
- added NT4: NetTie_2, NetTie:NetTie-2_SMD_Pad2.0mm, B.Cu at (150.9, 72.4)
- added R38: 10K 1% 0805, Resistor_SMD:R_0805_2012Metric_Pad1.20x1.40mm_HandSolder, F.Cu at (183.3, 90.2)
- added R39: 10K 1% 0805, Resistor_SMD:R_0805_2012Metric_Pad1.20x1.40mm_HandSolder, F.Cu at (183.3, 92.7)
- added R55: 10K 1% 0805, Resistor_SMD:R_0805_2012Metric_Pad1.20x1.40mm_HandSolder, F.Cu at (187.8, 90.2)
- added R56: 10K 1% 0805, Resistor_SMD:R_0805_2012Metric_Pad1.20x1.40mm_HandSolder, F.Cu at (187.8, 92.7)
- C15: value 1000uF 100V Electrolytic D18 -> 22uF 100V Electrolytic; footprint Capacitor_THT:CP_Radial_D18.0mm_P7.50mm -> Capacitor_THT:CP_Radial_D6.3mm_P2.50mm
- L1, L2: value Aprox 220uH -> Aprox 1mH; footprint Inductor_THT:L_Toroid_Vertical_L25.4mm_W14.7mm_P12.20mm_Vishay_TJ5_BigPads -> Inductor_THT:L_Toroid_Vertical_L31.8mm_W15.9mm_P13.50mm_Bourns_5700
- NT1, NT2: footprint NetTie:NetTie-2_SMD_Pad2.0mm -> NetTie:NetTie-2_SMD_Pad0.5mm
- moved L2 88.6 mm to (161.7, 67.7)
- moved C16 87.6 mm to (149.4, 121.5), turned to 90 degrees
- moved Q2 87.2 mm to (156.7, 126.0), turned to 180 degrees
- moved J13 85.9 mm to (137.7, 115.5), turned to 180 degrees
- moved C17 84.4 mm to (153.0, 83.5), turned to 90 degrees
- moved R27 77.6 mm to (155.8, 121.0), turned to 0 degrees
- moved D16 71.7 mm to (185.2, 64.0), turned to -90 degrees
- moved J3 69.2 mm to (205.7, 96.8)
- moved R25 65.9 mm to (189.7, 97.0), turned to 180 degrees
- moved J4 64.6 mm to (206.0, 66.0)
- moved NT1 62.6 mm to (190.9, 100.0), turned to -90 degrees
- moved NT2 62.6 mm to (188.4, 100.0), turned to -90 degrees
- moved J14 61.5 mm to (190.9, 103.3), turned to -90 degrees
- moved C15 61.3 mm to (196.0, 66.0), turned to -90 degrees
- moved J11 58.4 mm to (110.5, 66.5), turned to 0 degrees
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Connections:
- net Net-(K1-Pad1) renamed /SepicConverter/V_Bleed
- C14 pad 2: Net-(D4-A) -> Net-(C14-Pad2)
- D16 pad 1: /AnalogConverters/VIN -> Net-(C14-Pad2)
- D16 pad 2: GNDPWR -> /AnalogConverters/VOUT
- D16 pad 3: (no net) -> Net-(C14-Pad2)
- D4 pad 1: /AnalogConverters/VOUT -> GNDPWR
- D4 pad 2: Net-(D4-A) -> /AnalogConverters/VIN
- D4 pad 3: (no net) -> GNDPWR
- J12 pad 2: GNDPWR -> GNDA
- L2 pad 1: Net-(D4-A) -> Net-(C14-Pad2)
- NT3 pad 1: GNDPWR -> GNDA
- NT3 pad 2: GNDA -> GNDPWR
Routing:
- net +3.3V: track 95.8 -> 433.7 mm, vias 28 -> 31
- net GNDA: track 129.9 -> 436.9 mm, vias 54 -> 354
- net +12V: track 18.7 -> 168.1 mm, vias 0 -> 2
- net /AnalogConverters/VIN: track 3.14 -> 141.2 mm, vias 1 -> 20
- net /AnalogConverters/Isense+: track 6.13 -> 139.5 mm, vias 1 -> 2
- net /AnalogConverters/Isense-: track 11.0 -> 142.6 mm, vias 1 -> 2
- net /AnalogConverters/VOUT: track 0.00 -> 104.0 mm, vias 0 -> 14
- net /Pico/Tracer_En: track 12.0 -> 98.7 mm, vias 0 -> 2
- net /Pico/Tracer_pwm: track 12.0 -> 98.5 mm, vias 0 -> 2
- net Net-(Q2-D): track 0.00 -> 74.5 mm, vias 0 -> 1
- net Net-(Q3-G): track 0.00 -> 71.9 mm, vias 0 -> 1
- net /AnalogConverters/ADC_Input_Curr: track 0.00 -> 70.2 mm, vias 0 -> 2
- net /AnalogConverters/VPWR: track 0.00 -> 67.8 mm
- net /AnalogConverters/DRDY_PT100: track 0.00 -> 67.1 mm
- net /AnalogConverters/INA_OOR_Alert: track 3.25 -> 66.0 mm
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- added copper zone on B.Cu, net GNDA
- added copper zone on F.Cu, net GNDA
- added copper zone on B.Cu, net GNDPWR
- added copper zone on F.Cu, net GNDPWR
Other:
- board outline added: 180 x 80 mm
- board text added: "+ GND"
- board text added: "+12V"
- board text added: "+3.3V"
- board text added: "- +"
- board text added: "0 Jumpers = 40W 1 Jumpers = 20W 2 Jumpers = 10W"
- board text added: "12V Disconnect"
- board text added: "12V IN"
- board text added: "2W"
- board text added: "3W"
- board text added: "3W | 2W"
- board text added: "BUCK Disconnect"
- board text added: "Blinky"
- board text added: "CS"
- board text added: "D12"
- board text added: "DEBUG"
- board text added: "Electronic Engineering Final Project, Group 10"
- board text added: "GATE"
- board text added: "GND"
- board text added: "GND VIN+"
- board text added: "GPIO0"
- board text added: "GPIO1"
- board text added: "GPIO4"
- board text added: "GPIO7"
- board text added: "GPIO8"
- board text added: "GPIO9"
- board text added: "I2C"
- board text added: "INT | USB"
- board text added: "ON"
- board text added: "PT100"
- board text added: "PT100 Wires:"
- board text added: "PWM_Gate"
- board text added: "Pico VDD"
- board text added: "RX"
- board text added: "SCK"
- board text added: "SCL"
- board text added: "SDA"
- board text added: "SENSE"
- board text added: "SPI1"
- board text added: "SWCLK"
- board text added: "SWDIO"
- board text added: "TX"
- board text added: "Tracer_En"
- board text added: "Tracer_pwm"
- board text added: "VIN SENSE"
- board text added: "VOUT"
- board text added: "VOUT SENSE"
- board text removed: "C4"
- board text removed: "JP6"
- board text removed: "JP7"
- board text removed: "JP9"
- board text removed: "R7"

Commit message: HW: Version 1.0
Parts:
- removed D14, D15, D7, D8: WS2812, LED_SMD:LED_WS2812_PLCC6_5.0x5.0mm_P1.6mm
- added C26: 2.2uF 100V 1206, Capacitor_SMD:C_1206_3216Metric, F.Cu at (151.1, 91.4)
- added C32: 2.2uF 100V 1206, Capacitor_SMD:C_1206_3216Metric, F.Cu at (151.1, 94.0)
- added C35: 2.2uF 100V 1206, Capacitor_SMD:C_1206_3216Metric, F.Cu at (151.1, 96.5)
- added C36: 2.2uF 100V 1206, Capacitor_SMD:C_1206_3216Metric, F.Cu at (151.2, 99.1)
- added C39: 2.2uF 100V 1206, Capacitor_SMD:C_1206_3216Metric, F.Cu at (151.1, 101.6)
- added C46: 2.2uF 100V 1206, Capacitor_SMD:C_1206_3216Metric, F.Cu at (151.1, 104.1)
- added D19: WS2812B, LED_SMD:LED_WS2812B_PLCC4_5.0x5.0mm_P3.2mm, F.Cu at (105.4, 97.8)
- added D20: WS2812B, LED_SMD:LED_WS2812B_PLCC4_5.0x5.0mm_P3.2mm, F.Cu at (116.8, 97.8)
- added D21: WS2812B, LED_SMD:LED_WS2812B_PLCC4_5.0x5.0mm_P3.2mm, F.Cu at (116.8, 106.7)
- added D22: WS2812B, LED_SMD:LED_WS2812B_PLCC4_5.0x5.0mm_P3.2mm, F.Cu at (105.4, 106.7)
- added J9: Barrel_Jack_MountingPin, Connector_BarrelJack:BarrelJack_GCT_DCJ200-10-A_Horizontal, F.Cu at (143.5, 64.4)
- added R57: 10K 1% 0805, Resistor_SMD:R_0805_2012Metric, F.Cu at (196.2, 79.4)
- added R58: 10K 1% 0805, Resistor_SMD:R_0805_2012Metric, F.Cu at (196.2, 74.3)
- C10, C13, C18, C19, C20, C21, C27, C28, C3, C33, C34, C4, C41, C43, C45, C5, C9: footprint Capacitor_SMD:C_0805_2012Metric_Pad1.18x1.45mm_HandSolder -> Capacitor_SMD:C_0805_2012Metric
- C16, C25: value 1nF 1KV X7R 1206 -> 1nF 10% 1KV X7R 1206; footprint Capacitor_SMD:C_1206_3216Metric_Pad1.33x1.80mm_HandSolder -> Capacitor_SMD:C_1206_3216Metric
- C22, C23, C24: footprint Capacitor_SMD:C_1210_3225Metric_Pad1.33x2.70mm_HandSolder -> Capacitor_SMD:C_1210_3225Metric
- C29, C30, C31: value C -> 100nF 10% 50V X7R 0805; footprint Capacitor_SMD:C_0805_2012Metric_Pad1.18x1.45mm_HandSolder -> Capacitor_SMD:C_0805_2012Metric
- C37, C38, C40, C42, C44, C6: footprint Capacitor_SMD:C_1206_3216Metric_Pad1.33x1.80mm_HandSolder -> Capacitor_SMD:C_1206_3216Metric
- D10, D13, D2, D3: value BAT54S -> BAT54SLT1G
- D11, D12, D6: value Red Led 0805 -> YLED0805 Red; footprint LED_SMD:LED_0805_2012Metric_Pad1.15x1.40mm_HandSolder -> LED_SMD:LED_0805_2012Metric
- D16, D4: value MBRB20200 -> MBRB20200CT
- D9: value BZX84C15 -> BZX84C15LT1G
- L1, L2: value Aprox 1mH -> 1mH 2.4A
- L3: value 2.2uH 3A -> XFL4020-222MEC
- Q1: value MMBT3904 -> MMBT3904LT1G
- R1, R3, R5, R8: value R_US -> 10K 1% 0805; footprint Resistor_SMD:R_0805_2012Metric_Pad1.20x1.40mm_HandSolder -> Resistor_SMD:R_0805_2012Metric
- R10, R11, R12, R13, R14, R15, R16, R17, R18, R19, R2, R20, R21, R22, R23, R24, R26, R28, R30, R31, R32, R33, R34, R35, R36, R37, R38, R39, R40, R41, R42, R43, R44, R45, R46, R47, R48, R49, R50, R51, R52, R53, R54, R55, R56, R7: footprint Resistor_SMD:R_0805_2012Metric_Pad1.20x1.40mm_HandSolder -> Resistor_SMD:R_0805_2012Metric
- R25, R27: footprint Resistor_SMD:R_2512_6332Metric_Pad1.40x3.35mm_HandSolder -> Resistor_SMD:R_2512_6332Metric
- R29: value 10m 3W 1% 2512 -> 100m 3W 1% 2512; footprint Resistor_SMD:R_2512_6332Metric_Pad1.40x3.35mm_HandSolder -> Resistor_SMD:R_2512_6332Metric
- R4: value R_US -> 2.7K 1% 0805; footprint Resistor_SMD:R_0805_2012Metric_Pad1.20x1.40mm_HandSolder -> Resistor_SMD:R_0805_2012Metric
- R6: value R_US -> 100R 1% 0805; footprint Resistor_SMD:R_0805_2012Metric_Pad1.20x1.40mm_HandSolder -> Resistor_SMD:R_0805_2012Metric
- SW1, SW2: value SW_SPST -> 1TS009A-1800-5000-CT
- U2: value INA229 -> INA229AIDGSR
- U3: value INA281A3 -> INA281A3IDBVR
- U4: value TC4422 -> TC4422ESM
- U5: value MCP601-xOT -> OPA171AIDBVR
- U8: value AP62250WU -> AP62250WU-7; footprint Package_TO_SOT_SMD:TSOT-23-6_HandSoldering -> Package_TO_SOT_SMD:TSOT-23-6
- moved G*** 84.9 mm to (128.3, 108.0)
- moved C14 54.5 mm to (151.1, 109.9), turned to 90 degrees
- moved K1 40.8 mm to (188.0, 85.7)
- moved D17 37.0 mm to (184.2, 80.6)
- moved C17 35.7 mm to (174.0, 112.4), turned to -90 degrees
- moved L1 22.8 mm to (176.5, 88.9), turned to -90 degrees
- moved R56 19.3 mm to (193.7, 74.3), turned to -90 degrees
- moved R39 16.9 mm to (193.7, 79.4), turned to -90 degrees
- moved R25 16.7 mm to (202.6, 86.4)
- moved NT2 16.6 mm to (201.3, 89.5)
- moved R55 16.2 mm to (191.1, 74.3), turned to -90 degrees
- moved J14 15.8 mm to (202.6, 92.7)
- moved NT1 15.3 mm to (202.6, 90.2)
- moved C16 13.6 mm to (162.6, 118.1)
- moved R38 13.3 mm to (191.1, 79.4), turned to -90 degrees
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Connections:
- C33 pad 1: +3.3V -> +12V
- C37 pad 1: +3.3V -> +12V
- J12 pad 1: Net-(D18-A1) -> +12V
- U5 pad 5: +3.3V -> +12V
Routing:
- net +12V: track 168.1 -> 236.6 mm, vias 2 -> 4
- net /AnalogConverters/VIN: track 141.2 -> 200.1 mm, vias 20 -> 19
- net /SepicConverter/V_Bleed: track 55.6 -> 3.95 mm
- net Net-(D14-DIN): track 47.0 -> 0.00 mm
- net /SepicConverter/Tracer_Coil: track 47.4 -> 90.3 mm, vias 0 -> 1
- net /SepicConverter/CurveTracer: track 14.4 -> 54.8 mm, vias 0 -> 1
- net /AnalogConverters/VPWR: track 67.8 -> 94.1 mm, vias 0 -> 1
- net +3.3V: track 433.7 -> 410.2 mm, vias 31 -> 30
- net Net-(C14-Pad2): track 48.0 -> 70.5 mm
- net Net-(D18-A1): track 25.5 -> 46.6 mm
- net Net-(D21-DOUT): track 0.00 -> 19.2 mm
- net Net-(D19-DOUT): track 0.00 -> 17.1 mm
- net Net-(D14-DOUT): track 17.1 -> 0.00 mm
- net Net-(D7-DOUT): track 15.5 -> 0.00 mm
- net Net-(Q2-D): track 74.5 -> 59.1 mm, vias 1 -> 0
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Other:
- board text added: "12V Disc"
- board text added: "3.3V"
- board text added: "BUCK Disc"
- board text added: "DC IN"
- board text added: "Electronic Engineering MPP_SDK V1.0 07/06/2026"
- board text added: "VIN"
- board text removed: "12V Disconnect"
- board text removed: "BUCK Disconnect"
- board text removed: "Electronic Engineering Final Project, Group 10"
- board text removed: "GND VIN+"
