File: hardware/Proyecto0.1V.kicad_pcb (KiCad board)
At the start: 2 copper layers, 121 parts, among them J1 Conn_01x03 2.54mm, J11 Conn_01x02, J12 Conn_01x02, J13 Conn_01x02, J14 Conn_01x02, J2 Conn_01x03 5.08mm, J3 Conn_01x04 5.08mm, J4 Conn_01x04 5.08mm, J5 Conn_01x04, J6 Conn_01x06, J7 Conn_01x12, Q2 IPP200N25N3, U1 MAX31865xTP, U10 SRV05-4, U2 INA229, U3 INA281A3, U4 TC4422, U6 SRV05-4, U7 SRV05-4, U8 AP62250WU, U9 SRV05-4

Commit message: Hw/placa sepic (#34)
Co-authored-by: Federico Borello <156438142+fborello-lambda@users.noreply.github.com>
Parts:
- removed C1, C11, C7: 1uF 10% 50V X7R 0805, Capacitor_SMD:C_0805_2012Metric_Pad1.18x1.45mm_HandSolder
- removed C12, C2, C8: 100nF 10% 100V X7R 0805, Capacitor_SMD:C_0805_2012Metric_Pad1.18x1.45mm_HandSolder
- removed D7, D8: Red Led 0805, LED_SMD:LED_0805_2012Metric_Pad1.15x1.40mm_HandSolder
- removed JP2, JP3, JP4, JP5: Jumper_2_Open, Connector_PinHeader_2.54mm:PinHeader_1x02_P2.54mm_Vertical
- added C13: 100nF 10% 50V X7R 0805, Capacitor_SMD:C_0805_2012Metric, F.Cu at (121.8, 98.0)
- added C18: 100nF 10% 50V X7R 0805, Capacitor_SMD:C_0805_2012Metric, F.Cu at (110.5, 97.6)
- added C20: 100nF 10% 50V X7R 0805, Capacitor_SMD:C_0805_2012Metric, F.Cu at (121.9, 106.7)
- added C21: 100nF 10% 50V X7R 0805, Capacitor_SMD:C_0805_2012Metric, F.Cu at (110.5, 106.7)
- added C29: 100nF 10% 50V X7R 0805, Capacitor_SMD:C_0805_2012Metric, F.Cu at (93.8, 122.4)
- added C30: 100nF 10% 50V X7R 0805, Capacitor_SMD:C_0805_2012Metric, F.Cu at (98.9, 124.9)
- added C31: 100nF 10% 50V X7R 0805, Capacitor_SMD:C_0805_2012Metric, F.Cu at (98.9, 114.8)
- added C32: 2.2uF 100V 1206, Capacitor_SMD:C_1206_3216Metric, F.Cu at (151.1, 94.0)
- added C33: 100nF 10% 50V X7R 0805, Capacitor_SMD:C_0805_2012Metric, F.Cu at (104.0, 117.3)
- added C34: 100nF 10% 50V X7R 0805, Capacitor_SMD:C_0805_2012Metric, F.Cu at (112.9, 118.6)
- added C35: 2.2uF 100V 1206, Capacitor_SMD:C_1206_3216Metric, F.Cu at (151.1, 96.5)
- added C36: 2.2uF 100V 1206, Capacitor_SMD:C_1206_3216Metric, F.Cu at (151.2, 99.1)
- added C37: 1uF 10% 100V X7R 1206, Capacitor_SMD:C_1206_3216Metric, F.Cu at (104.0, 114.8)
- added C38: 1uF 10% 100V X7R 1206, Capacitor_SMD:C_1206_3216Metric, F.Cu at (112.9, 114.8)
- added C39: 2.2uF 100V 1206, Capacitor_SMD:C_1206_3216Metric, F.Cu at (151.1, 101.6)
- added C40: 1uF 10% 100V X7R 1206, Capacitor_SMD:C_1206_3216Metric, F.Cu at (54.4, 114.8)
- added C41: 100nF 10% 50V X7R 0805, Capacitor_SMD:C_0805_2012Metric, F.Cu at (48.1, 116.0)
- added C42: 1uF 10% 100V X7R 1206, Capacitor_SMD:C_1206_3216Metric, F.Cu at (83.0, 123.7)
- added C43: 100nF 10% 50V X7R 0805, Capacitor_SMD:C_0805_2012Metric, F.Cu at (76.6, 123.7)
- added C44: 1uF 10% 100V X7R 1206, Capacitor_SMD:C_1206_3216Metric, F.Cu at (65.8, 124.9)
- added C45: 100nF 10% 50V X7R 0805, Capacitor_SMD:C_0805_2012Metric, F.Cu at (70.9, 123.7)
- added C46: 2.2uF 100V 1206, Capacitor_SMD:C_1206_3216Metric, F.Cu at (151.1, 104.1)
- added D16: MBRB20200CT, Package_TO_SOT_SMD:TO-263-2, F.Cu at (190.5, 59.1)
- added D17: SS110, Diode_SMD:D_SMA_Handsoldering, F.Cu at (184.2, 80.6)
- added D18: SMAJ14A, Diode_SMD:D_SMA, F.Cu at (135.3, 55.6)
- added D19: WS2812B, LED_SMD:LED_WS2812B_PLCC4_5.0x5.0mm_P3.2mm, F.Cu at (105.4, 97.8)
- added D20: WS2812B, LED_SMD:LED_WS2812B_PLCC4_5.0x5.0mm_P3.2mm, F.Cu at (116.8, 97.8)
- added D21: WS2812B, LED_SMD:LED_WS2812B_PLCC4_5.0x5.0mm_P3.2mm, F.Cu at (116.8, 106.7)
- added D22: WS2812B, LED_SMD:LED_WS2812B_PLCC4_5.0x5.0mm_P3.2mm, F.Cu at (105.4, 106.7)
- added G***: LOGO, Custom_Library:logo_Grupo, F.Cu at (128.3, 108.0)
- added G***: LOGO, Custom_Library:UTN_LOGO, F.Cu at (198.1, 124.5)
- added H1: MountingHole_Pad, MountingHole:MountingHole_3.2mm_M3_Pad, F.Cu at (204.7, 56.0)
- added H2: MountingHole_Pad, MountingHole:MountingHole_3.2mm_M3_Pad, F.Cu at (204.7, 122.0)
- added H3: MountingHole_Pad, MountingHole:MountingHole_3.2mm_M3_Pad, F.Cu at (39.0, 123.0)
- added H4: MountingHole_Pad, MountingHole:MountingHole_3.2mm_M3_Pad, F.Cu at (39.0, 57.0)
- added J8: Conn_01x04, Connector_PinHeader_2.54mm:PinHeader_1x04_P2.54mm_Vertical, F.Cu at (49.3, 76.7)
- added J9: Barrel_Jack_MountingPin, Connector_BarrelJack:BarrelJack_GCT_DCJ200-10-A_Horizontal, F.Cu at (143.5, 64.4)
- added JP13: Jumper_2_Open, Connector_PinHeader_2.54mm:PinHeader_1x02_P2.54mm_Vertical, F.Cu at (109.7, 83.6)
- added JP6: Jumper_2_Open, Connector_PinHeader_2.54mm:PinHeader_1x02_P2.54mm_Vertical, F.Cu at (132.5, 79.8)
- added K1: G5LE-1, Relay_THT:Relay_SPDT_Omron-G5LE-1, F.Cu at (188.0, 85.7)
- added NT4: NetTie_2, NetTie:NetTie-2_SMD_Pad2.0mm, B.Cu at (143.2, 69.0)
- added Q1: MMBT3904LT1G, Package_TO_SOT_SMD:SOT-23, F.Cu at (129.0, 94.2)
- added Q3: IPP200N25N3, Package_TO_SOT_THT:TO-220-3_Vertical, F.Cu at (148.6, 123.2)
- added R1: 10K 1% 0805, Resistor_SMD:R_0805_2012Metric, F.Cu at (93.8, 119.8)
- added R17: 75K 1% 0805, Resistor_SMD:R_0805_2012Metric, F.Cu at (117.3, 76.7)
- added R28: 4.7K 1% 0805, Resistor_SMD:R_0805_2012Metric, F.Cu at (62.0, 56.3)
- added R29: 100m 3W 1% 2512, Resistor_SMD:R_2512_6332Metric, F.Cu at (145.4, 117.5)
- added R3: 10K 1% 0805, Resistor_SMD:R_0805_2012Metric, F.Cu at (93.8, 124.9)
- added R30: 75K 1% 0805, Resistor_SMD:R_0805_2012Metric, F.Cu at (117.3, 79.2)
- added R37: 4.7K 1% 0805, Resistor_SMD:R_0805_2012Metric, F.Cu at (129.0, 98.0)
- added R38: 10K 1% 0805, Resistor_SMD:R_0805_2012Metric, F.Cu at (191.1, 79.4)
- added R54: 4.7K 1% 0805, Resistor_SMD:R_0805_2012Metric, F.Cu at (109.0, 57.6)
- added R55: 10K 1% 0805, Resistor_SMD:R_0805_2012Metric, F.Cu at (191.1, 74.3)
- added R56: 10K 1% 0805, Resistor_SMD:R_0805_2012Metric, F.Cu at (193.7, 74.3)
- added R57: 10K 1% 0805, Resistor_SMD:R_0805_2012Metric, F.Cu at (196.2, 79.4)
- added R58: 10K 1% 0805, Resistor_SMD:R_0805_2012Metric, F.Cu at (196.2, 74.3)
- added SW1: 1TS009A-1800-5000-CT, Button_Switch_SMD:SW_Push_1TS009xxxx-xxxx-xxxx_6x6x5mm, F.Cu at (54.8, 54.8)
- added SW2: 1TS009A-1800-5000-CT, Button_Switch_SMD:SW_Push_1TS009xxxx-xxxx-xxxx_6x6x5mm, F.Cu at (47.0, 54.8)
- added U5: OPA171AIDBVR, Package_TO_SOT_SMD:SOT-23-5, F.Cu at (98.9, 119.8)
- C10, C19, C27, C28, C3, C4, C5, C9: value 100nF 10% 100V X7R 0805 -> 100nF 10% 50V X7R 0805; footprint Capacitor_SMD:C_0805_2012Metric_Pad1.18x1.45mm_HandSolder -> Capacitor_SMD:C_0805_2012Metric
- C15: value 1000uF 100V Electrolytic D18 -> 22uF 100V Electrolytic; footprint Capacitor_THT:CP_Radial_D18.0mm_P7.50mm -> Capacitor_THT:CP_Radial_D6.3mm_P2.50mm
- C16: value 1nF 1000V -> 1nF 10% 1KV X7R 1206; footprint Capacitor_SMD:C_1210_3225Metric_Pad1.33x2.70mm_HandSolder -> Capacitor_SMD:C_1206_3216Metric
- C22: value 10uF 10% 50V X7R 0805 -> 22uF 10% 25V X7R 1210; footprint Capacitor_SMD:C_0805_2012Metric_Pad1.18x1.45mm_HandSolder -> Capacitor_SMD:C_1210_3225Metric
- C23: value 1uF 10% 50V X7R 0805 -> 22uF 10% 25V X7R 1210; footprint Capacitor_SMD:C_0805_2012Metric_Pad1.18x1.45mm_HandSolder -> Capacitor_SMD:C_1210_3225Metric
- C24: value 10uF 50V Aluminum Polymer -> 22uF 10% 25V X7R 1210; footprint Capacitor_THT:CP_Radial_D6.3mm_P2.50mm -> Capacitor_SMD:C_1210_3225Metric
- C25: value 3.3nF 10% 100V X7R 0805 -> 1nF 10% 1KV X7R 1206; footprint Capacitor_SMD:C_0805_2012Metric_Pad1.18x1.45mm_HandSolder -> Capacitor_SMD:C_1206_3216Metric
- C26: value 10uF 50V Aluminum Polymer -> 2.2uF 100V 1206; footprint Capacitor_THT:CP_Radial_D6.3mm_P2.50mm -> Capacitor_SMD:C_1206_3216Metric
- C6: value 1uF 10% 100V X7R 1210 -> 1uF 10% 100V X7R 1206; footprint Capacitor_SMD:C_1210_3225Metric_Pad1.33x2.70mm_HandSolder -> Capacitor_SMD:C_1206_3216Metric
- D1, D5: footprint Diode_SMD:D_SMA -> Diode_SMD:D_SMA_Handsoldering
- D10, D13, D2, D3: value BAT54S -> BAT54SLT1G
- D11, D12, D6: value Red Led 0805 -> YLED0805 Red; footprint LED_SMD:LED_0805_2012Metric_Pad1.15x1.40mm_HandSolder -> LED_SMD:LED_0805_2012Metric
- D4: value MBRB20200 -> MBRB20200CT
- D9: value BZX84C15 -> BZX84C15LT1G
- L1, L2: value Aprox 220uH -> 1mH 2.4A; footprint Inductor_THT:L_Toroid_Vertical_L25.4mm_W14.7mm_P12.20mm_Vishay_TJ5_BigPads -> Inductor_THT:L_Toroid_Vertical_L31.8mm_W15.9mm_P13.50mm_Bourns_5700
- L3: value 4.7uH 3A -> XFL4020-222MEC; footprint Inductor_SMD:L_12x12mm_H8mm -> Inductor_SMD_Wurth:L_Wurth_WE-LQSH-4020
- NT1, NT2: footprint NetTie:NetTie-2_SMD_Pad2.0mm -> NetTie:NetTie-2_SMD_Pad0.5mm
- R10, R11, R18, R19: value 10R 1% 0805 Resistor -> 10R 1% 0805; footprint Resistor_SMD:R_0805_2012Metric_Pad1.20x1.40mm_HandSolder -> Resistor_SMD:R_0805_2012Metric
- R12, R13, R14, R16: value R_US -> 75K 1% 0805; footprint Resistor_SMD:R_0805_2012Metric_Pad1.20x1.40mm_HandSolder -> Resistor_SMD:R_0805_2012Metric
- R15, R5, R7, R8: value R_US -> 10K 1% 0805; footprint Resistor_SMD:R_0805_2012Metric_Pad1.20x1.40mm_HandSolder -> Resistor_SMD:R_0805_2012Metric
- R2: value 400R 0.1% -> 400R 0.1% 0805; footprint Resistor_SMD:R_0805_2012Metric_Pad1.20x1.40mm_HandSolder -> Resistor_SMD:R_0805_2012Metric
- R20: value 33R 1% 0805 Resistor -> 33R 1% 0805; footprint Resistor_SMD:R_0805_2012Metric_Pad1.20x1.40mm_HandSolder -> Resistor_SMD:R_0805_2012Metric
- R21, R22: value 4.7Kohm -> 4.7K 1% 0805; footprint Resistor_SMD:R_0805_2012Metric_Pad1.20x1.40mm_HandSolder -> Resistor_SMD:R_0805_2012Metric
- R23: value 10K 1% 0805 Resistor -> 10K 1% 0805; footprint Resistor_SMD:R_0805_2012Metric_Pad1.20x1.40mm_HandSolder -> Resistor_SMD:R_0805_2012Metric
- R24, R40: value 150R -> 330R 1% 0805; footprint Resistor_SMD:R_0805_2012Metric_Pad1.20x1.40mm_HandSolder -> Resistor_SMD:R_0805_2012Metric
- R25: value 10mOhm 3W 1% 2512 -> 10m 3W 1% 2512; footprint Resistor_SMD:R_2512_6332Metric_Pad1.40x3.35mm_HandSolder -> Resistor_SMD:R_2512_6332Metric
- R26, R31: value 150R -> 4.7K 1% 0805; footprint Resistor_SMD:R_0805_2012Metric_Pad1.20x1.40mm_HandSolder -> Resistor_SMD:R_0805_2012Metric
- R27: value 4.7R Ohm 3W 1% 2512 -> 4.7R 3W 1% 2512; footprint Resistor_SMD:R_2512_6332Metric_Pad1.40x3.35mm_HandSolder -> Resistor_SMD:R_2512_6332Metric
- R32: value 10R 1% -> 33R 1% 0805; footprint Resistor_SMD:R_0805_2012Metric_Pad1.20x1.40mm_HandSolder -> Resistor_SMD:R_0805_2012Metric
- R33, R34, R35, R36, R41, R42, R43, R44, R45, R46: value 330R 1% -> 330R 1% 0805; footprint Resistor_SMD:R_0805_2012Metric_Pad1.20x1.40mm_HandSolder -> Resistor_SMD:R_0805_2012Metric
- R39: value 1K 1206 -> 10K 1% 0805; footprint Resistor_SMD:R_0805_2012Metric_Pad1.20x1.40mm_HandSolder -> Resistor_SMD:R_0805_2012Metric
- R4: value R_US -> 2.7K 1% 0805; footprint Resistor_SMD:R_0805_2012Metric_Pad1.20x1.40mm_HandSolder -> Resistor_SMD:R_0805_2012Metric
- R47: value 33K 0805 -> 33R 1% 0805; footprint Resistor_SMD:R_0805_2012Metric_Pad1.20x1.40mm_HandSolder -> Resistor_SMD:R_0805_2012Metric
- R48, R49, R50, R51: value 33R 1% -> 33R 1% 0805; footprint Resistor_SMD:R_0805_2012Metric_Pad1.20x1.40mm_HandSolder -> Resistor_SMD:R_0805_2012Metric
- R52: value 10K 0805 -> 4.7K 1% 0805; footprint Resistor_SMD:R_0805_2012Metric_Pad1.20x1.40mm_HandSolder -> Resistor_SMD:R_0805_2012Metric
- R53: value 100K 0805 -> 100K 1% 0805; footprint Resistor_SMD:R_0805_2012Metric_Pad1.20x1.40mm_HandSolder -> Resistor_SMD:R_0805_2012Metric
- R6: value R_US -> 100R 1% 0805; footprint Resistor_SMD:R_0805_2012Metric_Pad1.20x1.40mm_HandSolder -> Resistor_SMD:R_0805_2012Metric
- U2: value INA229 -> INA229AIDGSR
- U3: value INA281A3 -> INA281A3IDBVR
- U4: value TC4422 -> TC4422ESM
- U8: value AP62250WU -> AP62250WU-7
- moved Q2 215.4 mm to (160.7, 123.2), turned to 180 degrees
- moved R27 210.0 mm to (156.8, 117.5), turned to 180 degrees
- moved C16 202.5 mm to (162.6, 118.1)
- moved C17 192.2 mm to (174.0, 112.4), turned to -90 degrees
- moved C14 189.9 mm to (151.1, 109.9), turned to 90 degrees
- moved L2 177.7 mm to (166.1, 67.9), turned to 180 degrees
- moved C5 170.6 mm to (70.9, 118.6), turned to 180 degrees
- moved R11 170.0 mm to (70.9, 121.1), turned to 180 degrees
- moved D11 169.9 mm to (109.0, 62.1), turned to 90 degrees
- moved U2 169.7 mm to (63.3, 119.8)
- moved R10 169.4 mm to (70.9, 116.0), turned to 180 degrees
- moved R5 168.6 mm to (93.8, 114.8), turned to 0 degrees
- moved R4 168.1 mm to (104.0, 124.9)
- moved R6 167.4 mm to (93.8, 117.3), turned to 0 degrees
- moved C6 165.2 mm to (65.8, 114.8), turned to 180 degrees
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Connections:
- net /Pico/GPIO2 renamed /Pico/Tracer_pwm
- net /Pico/GPIO5 renamed /Pico/GPIO8
- net /Pico/GPIO6 renamed /Pico/GPIO9
- A1 pad 1: /Pico/LED1 -> /Pico/But1
- A1 pad 10: /Pico/GPIO4 -> /Pico/GPIO7
- A1 pad 2: /Pico/LED2 -> /Pico/But2
- A1 pad 4: /Pico/GPIO1 -> /Pico/Tracer_En
- A1 pad 6: /Pico/GPIO3 -> /Pico/GPIO4
- C14 pad 2: Net-(D4-A) -> Net-(C14-Pad2)
- C23 pad 1: +12V -> +3.3V
- C23 pad 2: GNDPWR -> GNDA
- C24 pad 1: +12V -> +3.3V
- C24 pad 2: GNDPWR -> GNDA
- C26 pad 1: +3.3V -> Net-(Q2-D)
- C26 pad 2: GNDA -> Net-(C14-Pad2)
- C6 pad 1: /AnalogConverters/VPWR -> /AnalogConverters/VIN
- D4 pad 1: /AnalogConverters/VOUT -> GNDPWR
- D4 pad 2: Net-(D4-A) -> /AnalogConverters/VIN
- D4 pad 3: (no net) -> GNDPWR
- J12 pad 1: Net-(J12-Pin_1) -> +12V
- J12 pad 2: GNDPWR -> GNDA
- J3 pad 1: /SepicConverter/VIN -> /AnalogConverters/VIN
- J3 pad 2: /SepicConverter/VIN -> /AnalogConverters/VIN
- JP10 pad 1: /AnalogConverters/ADC_VOUT -> Net-(JP10-A)
- JP10 pad 2: Net-(JP10-B) -> /AnalogConverters/VOUT
- JP16 pad 2: Net-(J12-Pin_1) -> Net-(D18-A1)
- JP7 pad 1: /AnalogConverters/ADC_VOUT -> Net-(JP7-A)
- JP7 pad 2: Net-(JP7-B) -> Net-(JP6-A)
- JP8 pad 1: /AnalogConverters/ADC_VOUT -> Net-(JP13-B)
- JP8 pad 2: Net-(JP8-B) -> Net-(JP10-A)
- JP9 pad 1: /AnalogConverters/ADC_VOUT -> Net-(JP6-B)
- JP9 pad 2: Net-(JP9-B) -> /AnalogConverters/VPWR
- L2 pad 1: Net-(D4-A) -> Net-(C14-Pad2)
- NT1 pad 1: /SepicConverter/VIN -> /AnalogConverters/VIN
- NT2 pad 1: /AnalogConverters/VPWR -> /SepicConverter/V_Bleed
- NT3 pad 1: GNDPWR -> GNDA
- NT3 pad 2: GNDA -> GNDPWR
- R12 pad 1: /AnalogConverters/VOUT -> Net-(JP6-A)
- R12 pad 2: Net-(JP7-B) -> Net-(JP7-A)
- R13 pad 1: /AnalogConverters/VOUT -> Net-(JP6-B)
- R13 pad 2: Net-(JP8-B) -> Net-(JP6-A)
- R14 pad 1: /AnalogConverters/VOUT -> Net-(JP7-A)
- R14 pad 2: Net-(JP9-B) -> /AnalogConverters/ADC_VPWR
- R16 pad 1: /AnalogConverters/VOUT -> Net-(JP10-A)
- R16 pad 2: Net-(JP10-B) -> Net-(JP13-B)
- R25 pad 1: /SepicConverter/VIN -> /AnalogConverters/VIN
- R25 pad 2: /AnalogConverters/VPWR -> /SepicConverter/V_Bleed
- R26 pad 1: /Pico/LED1 -> +3.3V
- R26 pad 2: Net-(D7-A) -> /Pico/But2
- R31 pad 1: /Pico/LED2 -> Net-(Q1-B)
- R31 pad 2: Net-(D8-A) -> /Pico/Tracer_En
- R33 pad 1: /Pico/LED1 -> /Pico/But1
- R34 pad 1: /Pico/LED2 -> /Pico/But2
- R35 pad 1: /Pico/GPIO1 -> /Pico/Tracer_En
- R39 pad 1: +12V -> Net-(R39-Pad1)
- R39 pad 2: Net-(D11-A) -> /SepicConverter/V_Bleed
- R4 pad 1: /AnalogConverters/VPWR -> GNDA
- R41 pad 1: /Pico/GPIO3 -> /Pico/GPIO4
- R42 pad 1: /Pico/GPIO4 -> /Pico/GPIO7
- R5 pad 1: /AnalogConverters/VPWR -> GNDA
- R5 pad 2: Net-(JP3-B) -> Net-(C31-Pad1)
- R6 pad 1: /AnalogConverters/VPWR -> Net-(Q3-G)
- R6 pad 2: Net-(JP4-B) -> Net-(C31-Pad1)
- R8 pad 1: /AnalogConverters/VPWR -> Net-(Q3-S)
- U10 pad 1: /Pico/OUT_SCK -> /Pico/OUT_TX
- U10 pad 3: /Pico/OUT_TX -> /Pico/OUT_SCK
- U10 pad 4: /Pico/OUT_RX -> /Pico/OUT_CS
- U10 pad 6: /Pico/OUT_CS -> /Pico/OUT_RX
- U2 pad 8: /AnalogConverters/VPWR -> /AnalogConverters/VIN
- U6 pad 1: /Pico/Out1 -> /Pico/Out2
- U6 pad 3: /Pico/Out2 -> /Pico/Out1
- U6 pad 4: /Pico/Out3 -> /Pico/Out4
- U6 pad 6: /Pico/Out4 -> /Pico/Out3
- U7 pad 1: /Pico/Out5 -> /Pico/Out6
- U7 pad 3: /Pico/Out6 -> /Pico/Out5
- U7 pad 4: /Pico/Out7 -> /Pico/Out8
- U7 pad 6: /Pico/Out8 -> /Pico/Out7
- U9 pad 1: /Pico/Out9 -> /Pico/I2C_SCL
- U9 pad 3: /Pico/Out10 -> /Pico/I2C_SDA
- U9 pad 4: /Pico/I2C_SDA -> /Pico/Out10
- U9 pad 6: /Pico/I2C_SCL -> /Pico/Out9
Routing:
- net GNDA: track 0.00 -> 431.6 mm, vias 0 -> 351
- net +3.3V: track 0.00 -> 410.2 mm, vias 0 -> 30
- net +12V: track 0.00 -> 236.6 mm, vias 0 -> 4
- net /AnalogConverters/VIN: track 0.00 -> 200.1 mm, vias 0 -> 19
- net /AnalogConverters/Isense-: track 0.00 -> 152.0 mm, vias 0 -> 3
- net /AnalogConverters/Isense+: track 0.00 -> 147.6 mm, vias 0 -> 3
- net /AnalogConverters/VOUT: track 0.00 -> 102.3 mm, vias 0 -> 16
- net /Pico/PWM_Gate: track 0.00 -> 99.0 mm, vias 0 -> 4
- net /Pico/Tracer_En: track 0.00 -> 98.7 mm, vias 0 -> 2
- net /Pico/Tracer_pwm: track 0.00 -> 98.5 mm, vias 0 -> 2
- net /AnalogConverters/VPWR: track 0.00 -> 94.1 mm, vias 0 -> 1
- net /SepicConverter/Tracer_Coil: track 0.00 -> 90.3 mm, vias 0 -> 1
- net /SepicConverter/Gate: track 0.00 -> 80.5 mm
- net Net-(Q3-G): track 0.00 -> 78.0 mm, vias 0 -> 1
- net /AnalogConverters/SPI_MOSI: track 0.00 -> 72.1 mm, vias 0 -> 2
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- added copper zone on B.Cu, net GNDA
- added copper zone on F.Cu, net GNDA
- added copper zone on B.Cu, net GNDPWR
- added copper zone on F.Cu, net GNDPWR
Other:
- board outline added: 180 x 80 mm
- board text added: "+ GND"
- board text added: "+12V"
- board text added: "+3.3V"
- board text added: "- +"
- board text added: "0 Jumpers = 40W 1 Jumpers = 20W 2 Jumpers = 10W"
- board text added: "12V Disc"
- board text added: "12V IN"
- board text added: "2W"
- board text added: "3.3V"
- board text added: "3W"
- board text added: "3W | 2W"
- board text added: "BUCK Disc"
- board text added: "Blinky"
- board text added: "CS"
- board text added: "D12"
- board text added: "DC IN"
- board text added: "DEBUG"
- board text added: "Electronic Engineering MPP_SDK V1.0 07/06/2026"
- board text added: "GATE"
- board text added: "GND"
- board text added: "GPIO0"
- board text added: "GPIO1"
- board text added: "GPIO4"
- board text added: "GPIO7"
- board text added: "GPIO8"
- board text added: "GPIO9"
- board text added: "I2C"
- board text added: "INT | USB"
- board text added: "ON"
- board text added: "PT100"
- board text added: "PT100 Wires:"
- board text added: "PWM_Gate"
- board text added: "Pico VDD"
- board text added: "RX"
- board text added: "SCK"
- board text added: "SCL"
- board text added: "SDA"
- board text added: "SENSE"
- board text added: "SPI1"
- board text added: "SWCLK"
- board text added: "SWDIO"
- board text added: "TX"
- board text added: "Tracer_En"
- board text added: "Tracer_pwm"
- board text added: "VIN"
- board text added: "VIN SENSE"
- board text added: "VOUT"
- board text added: "VOUT SENSE"
