File: hardware/SepicConverter.kicad_sch (KiCad schematic)
At the start: 11 parts, among them J3 Conn_01x04 5.08mm, J4 Conn_01x04 5.08mm, Q1 IRF640N, U4 TC4422

Commit message: HW: sch near final version
Parts:
- added NT1, NT2: NetTie_2, NetTie:NetTie-2_SMD_Pad2.0mm, symbol Device:NetTie_2
- added R25: 10mOhm 3W 1% 2512, Resistor_SMD:R_2512_6332Metric_Pad1.40x3.35mm_HandSolder, symbol Device:R_US
Connections:
- net VNEGP is gone; now on net GNDPWR: C13.2, C15.1, J3.3 (Pin_3), J3.4 (Pin_4), J4.3 (Pin_3), J4.4 (Pin_4), L2.2, Q1.S
- net VIN: now also NT1.1, R25.1; no longer C13.1, L1.1
- net VNEGA renamed GNDPWR
- net VOUT renamed Vout
- net Vgate renamed Gate
- net Vusb renamed +12V
- new net Isense+: NT1.2
- new net Isense-: NT2.2
- new net VPWR: C13.1, L1.1, NT2.1, R25.2

Commit message: HW: Sch done. PCB WIP
Parts:
- removed C13, C15: 1000uF 100V Electrolytic D18, Capacitor_THT:CP_Radial_D18.0mm_P7.50mm, symbol Device:C
- removed Q1: IRF640N, Package_TO_SOT_THT:TO-220-3_Horizontal_TabDown, symbol Device:Q_NMOS
- added C15, C17: 1000uF 100V Electrolytic D18, Capacitor_THT:CP_Radial_D18.0mm_P7.50mm, symbol Device:C_Polarized
- added C16: 1nF 1000V, symbol Device:C
- added C23: 1uF 10% 50V X7R 0805, Capacitor_SMD:C_0805_2012Metric_Pad1.18x1.45mm_HandSolder, symbol Device:C
- added C24: 10uF 50V Aluminum Polymer, Capacitor_THT:CP_Radial_D6.3mm_P2.50mm, symbol Device:C_Polarized
- added D1, D5: SS110, Diode_SMD:D_SMA, symbol Diode:SS110
- added D9: BZX84C15, Package_TO_SOT_SMD:SOT-23, symbol Diode:BZX84Cxx
- added J13, J14: Conn_01x02, Connector_PinHeader_2.54mm:PinHeader_1x02_P2.54mm_Vertical, symbol Connector_Generic:Conn_01x02
- added Q2: IPP200N25N3, Package_TO_SOT_THT:TO-220-3_Vertical, symbol Transistor_FET:IPP060N06N
- added R23: 10K 1% 0805 Resistor, Resistor_SMD:R_0805_2012Metric_Pad1.20x1.40mm_HandSolder, symbol Device:R_US
- added R27: 4.7R Ohm 3W 1% 2512, Resistor_SMD:R_2512_6332Metric_Pad1.40x3.35mm_HandSolder, symbol Device:R_US
- D4: value MBR10200 -> MBRB20200; footprint Package_TO_SOT_THT:TO-220F-3_Horizontal_TabDown -> Package_TO_SOT_SMD:TO-263-2; LCSC Part C5795369 -> C3011045; now in the parts list
- R20: value 10R 1% 0805 Resistor -> 33R 1% 0805 Resistor
Connections:
- net +12V: now also C23.1, C24.1, D1.1 (K)
- net GNDPWR: now also C15.2, C16.1, C17.2, C23.2, C24.2, D5.2 (A), D9.1 (A), J13.2 (Pin_2), Q2.3 (S), R23.1
- net Gate: now also D1.2 (A), D5.1 (K), D9.3 (K), J13.1 (Pin_1), Q2.1 (G), R23.2
- net Isense+: now also J14.1 (Pin_1)
- net Isense-: now also J14.2 (Pin_2)
- net VPWR: now also C17.1
- net Vout: now also C15.1
- net at C14.1, L1.2: now also Q2.2 (D), R27.2
- new net: C16.2, R27.1
Other:
- moved on the sheet: C14, D4, J3, J4, L1, L2, R25

Commit message: HW: Changes in GPIO components. PCB WIP
Changed lines of the file:
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@@
 		)
 		(property "Value" "1nF 1000V"
-			(at 157.988 59.69 0)
+			(at 152.654 60.452 0)
 			(show_name no)
 			(do_not_autoplace no)
@@
 		)
 		(property "Value" "1000uF 100V Electrolytic D18"
-			(at 176.276 58.166 0)
+			(at 169.164 59.436 0)
 			(show_name no)
 			(do_not_autoplace no)
@@
 		)
 		(property "Value" "1000uF 100V Electrolytic D18"
-			(at 120.396 58.166 0)
-			(show_name no)
-			(do_not_autoplace no)
+			(at 105.918 55.372 0)
+			(show_name no)
+			(do_not_autoplace no)

Commit message: HW: PCB WIP
Parts:
- removed C23: 1uF 10% 50V X7R 0805, Capacitor_SMD:C_0805_2012Metric_Pad1.18x1.45mm_HandSolder, symbol Device:C
- removed C24: 10uF 50V Aluminum Polymer, Capacitor_THT:CP_Radial_D6.3mm_P2.50mm, symbol Device:C_Polarized
- added C29, C30, C31: C, Capacitor_SMD:C_0805_2012Metric_Pad1.18x1.45mm_HandSolder, symbol Device:C
- added C33, C34: 100nF 10% 50V X7R 0805, Capacitor_SMD:C_0805_2012Metric_Pad1.18x1.45mm_HandSolder, symbol Device:C
- added C37, C38: 1uF 10% 100V X7R 1206, Capacitor_SMD:C_1206_3216Metric_Pad1.33x1.80mm_HandSolder, symbol Device:C
- added D16: MBRB20200, Package_TO_SOT_SMD:TO-263-2, symbol Device:D
- added D17: SS110, Diode_SMD:D_SMA_Handsoldering, symbol Diode:SS110
- added K1: G5LE-1, Relay_THT:Relay_SPDT_Omron-G5LE-1, symbol Relay:G5LE-1
- added Q1: MMBT3904, Package_TO_SOT_SMD:SOT-23, symbol Transistor_BJT:MMBT3904
- added Q3: IPP200N25N3, Package_TO_SOT_THT:TO-220-3_Vertical, symbol Transistor_FET:IPP060N06N
- added R1, R3, R4, R5, R6, R8: R_US, Resistor_SMD:R_0805_2012Metric_Pad1.20x1.40mm_HandSolder, symbol Device:R_US
- added R29: 10m 3W 1% 2512, Resistor_SMD:R_2512_6332Metric_Pad1.40x3.35mm_HandSolder, symbol Device:R_US
- added R31, R37: 4.7K 1% 0805, Resistor_SMD:R_0805_2012Metric_Pad1.20x1.40mm_HandSolder, symbol Device:R_US
- added U5: MCP601-xOT, Package_TO_SOT_SMD:SOT-23-5, symbol Amplifier_Operational:MCP601-xOT
- C15, C17: now left out of the parts list
- C16: value 1nF 1000V -> 1nF 1KV X7R 1206; footprint (none) -> Capacitor_SMD:C_1206_3216Metric_Pad1.33x1.80mm_HandSolder; now in the parts list
- D1, D5: footprint Diode_SMD:D_SMA -> Diode_SMD:D_SMA_Handsoldering
- R20: value 33R 1% 0805 Resistor -> 33R 1% 0805; LCSC Part C2907220 -> (none)
- R23: value 10K 1% 0805 Resistor -> 10K 1% 0805; LCSC Part C2907220 -> (none)
- R25: value 10mOhm 3W 1% 2512 -> 10m 3W 1% 2512
- R27: value 4.7R Ohm 3W 1% 2512 -> 4.7R 3W 1% 2512
Connections:
- net +12V: now also C34.1, C38.1, D17.1 (K), K1.2
- net GNDPWR: now also C34.2, C38.2, D16.2 (A), Q1.2 (E), R29.1
- net VIN: now also D16.1 (K)
- net VPWR: now also K1.4; no longer NT2.1, R25.2
- net Vout renamed VOUT
- new net: Q3.3 (S), R29.2, R8.1
- new net: C29.1, R1.2, R3.1
- new net: K1.1, NT2.1, R25.2
- new net: Q3.1 (G), R6.1
- new net: C31.1, R5.2, R6.2, U5.1
- new net: Q1.1 (B), R31.1, R37.1
- new net: C31.2, R8.2, U5.4 (-)
- new net: C30.1, R3.2, R4.2, U5.3 (+)
- new net +3.3V: C33.1, C37.1, U5.5 (V+)
- new net CurveTracer: K1.3, Q3.2 (D)
- new net GNDA: C29.2, C30.2, C33.2, C37.2, R4.1, R5.1, U5.2 (V-)
- new net Tracer_Coil: D17.2 (A), K1.5, Q1.3 (C)
- new net Tracer_En: R31.2, R37.2
- new net Tracer_pwm: R1.1
Other:
- moved on the sheet: C14, C15, C16, C17, D1, D4, D5, D9, J13, J14, J3, J4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

Commit message: HW: PCB Done
Parts:
- removed D16, D4: MBRB20200, Package_TO_SOT_SMD:TO-263-2, symbol Device:D
- added D16, D4: MBRB20200, Package_TO_SOT_SMD:TO-263-2, symbol Device:D_Schottky_Dual_CommonCathode_AKA_Parallel
- added R38, R39, R55, R56: 10K 1% 0805, Resistor_SMD:R_0805_2012Metric_Pad1.20x1.40mm_HandSolder, symbol Device:R_US
- C15: value 1000uF 100V Electrolytic D18 -> 22uF 100V Electrolytic; footprint Capacitor_THT:CP_Radial_D18.0mm_P7.50mm -> Capacitor_THT:CP_Radial_D6.3mm_P2.50mm
- L1, L2: value Aprox 220uH -> Aprox 1mH; footprint Inductor_THT:L_Toroid_Vertical_L25.4mm_W14.7mm_P12.20mm_Vishay_TJ5_BigPads -> Inductor_THT:L_Toroid_Vertical_L31.8mm_W15.9mm_P13.50mm_Bourns_5700
- NT1, NT2: footprint NetTie:NetTie-2_SMD_Pad2.0mm -> NetTie:NetTie-2_SMD_Pad0.5mm
Connections:
- net GNDPWR: now also D4.1 (A), D4.3 (A), R55.1, R56.1
- net VIN: now also D4.2 (K)
- net VOUT: now also D16.2 (K)
- net at C14.2, L2.1: now also D16.1 (A), D16.3 (A)
- net V_Bleed: now reaches K1.1, NT2.1, R25.2
- net V_Bleed: now also R38.2, R39.2
- new net: R38.1, R55.2
- new net: R39.1, R56.2

Commit message: HW: Version 1.0
Parts:
- added C26, C32, C35, C36, C39, C46: 2.2uF 100V 1206, Capacitor_SMD:C_1206_3216Metric, symbol Device:C
- added R57, R58: 10K 1% 0805, Resistor_SMD:R_0805_2012Metric, symbol Device:R_US
- C14: LCSC Part C5116053 -> (none)
- C15, C17: LCSC Part C3445915 -> (none)
- C16: value 1nF 1KV X7R 1206 -> 1nF 10% 1KV X7R 1206; footprint Capacitor_SMD:C_1206_3216Metric_Pad1.33x1.80mm_HandSolder -> Capacitor_SMD:C_1206_3216Metric
- C29, C30, C31: value C -> 100nF 10% 50V X7R 0805; footprint Capacitor_SMD:C_0805_2012Metric_Pad1.18x1.45mm_HandSolder -> Capacitor_SMD:C_0805_2012Metric
- C33, C34: footprint Capacitor_SMD:C_0805_2012Metric_Pad1.18x1.45mm_HandSolder -> Capacitor_SMD:C_0805_2012Metric
- C37, C38: footprint Capacitor_SMD:C_1206_3216Metric_Pad1.33x1.80mm_HandSolder -> Capacitor_SMD:C_1206_3216Metric
- D16, D4: value MBRB20200 -> MBRB20200CT; LCSC Part (none) -> C3874012
- D9: value BZX84C15 -> BZX84C15LT1G; LCSC Part (none) -> C80857
- J3, J4: LCSC Part C8446 -> (none)
- L1, L2: value Aprox 1mH -> 1mH 2.4A
- Q1: value MMBT3904 -> MMBT3904LT1G; LCSC Part (none) -> C81464
- Q2, Q3: now left out of the parts list
- R1, R3, R5, R8: value R_US -> 10K 1% 0805; footprint Resistor_SMD:R_0805_2012Metric_Pad1.20x1.40mm_HandSolder -> Resistor_SMD:R_0805_2012Metric
- R20, R23, R31, R37, R38, R39, R55, R56: footprint Resistor_SMD:R_0805_2012Metric_Pad1.20x1.40mm_HandSolder -> Resistor_SMD:R_0805_2012Metric
- R25, R27: footprint Resistor_SMD:R_2512_6332Metric_Pad1.40x3.35mm_HandSolder -> Resistor_SMD:R_2512_6332Metric
- R29: value 10m 3W 1% 2512 -> 100m 3W 1% 2512; footprint Resistor_SMD:R_2512_6332Metric_Pad1.40x3.35mm_HandSolder -> Resistor_SMD:R_2512_6332Metric
- R4: value R_US -> 2.7K 1% 0805; footprint Resistor_SMD:R_0805_2012Metric_Pad1.20x1.40mm_HandSolder -> Resistor_SMD:R_0805_2012Metric
- R6: value R_US -> 100R 1% 0805; footprint Resistor_SMD:R_0805_2012Metric_Pad1.20x1.40mm_HandSolder -> Resistor_SMD:R_0805_2012Metric
- U4: value TC4422 -> TC4422ESM
- U5: value MCP601-xOT -> OPA171AIDBVR; LCSC Part (none) -> C88036
Connections:
- net +3.3V is gone; now on net +12V: C33.1, C37.1, U5.5 (V+)
- net GNDPWR: now also R58.1
- net V_Bleed: now also R57.2
- net at C14.1, L1.2, Q2.2 (D)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: now also C26.1, C32.1, C35.1, C36.1, C39.1, C46.1
- net at C14.2, D16.1 (A), D16.3 (A)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: now also C26.2, C32.2, C35.2, C36.2, C39.2, C46.2
- new net: R57.1, R58.2
