File: hardware/SepicConverter.kicad_sch (KiCad schematic)
At the start: 24 parts, among them J13 Conn_01x02, J14 Conn_01x02, J3 Conn_01x04 5.08mm, J4 Conn_01x04 5.08mm, Q2 IPP200N25N3, U4 TC4422

Commit message: Hw/placa sepic (#34)
Co-authored-by: Federico Borello <156438142+fborello-lambda@users.noreply.github.com>
Parts:
- removed C23: 1uF 10% 50V X7R 0805, Capacitor_SMD:C_0805_2012Metric_Pad1.18x1.45mm_HandSolder, symbol Device:C
- removed C24: 10uF 50V Aluminum Polymer, Capacitor_THT:CP_Radial_D6.3mm_P2.50mm, symbol Device:C_Polarized
- removed D4: MBRB20200, Package_TO_SOT_SMD:TO-263-2, symbol Device:D
- added C26, C32, C35, C36, C39, C46: 2.2uF 100V 1206, Capacitor_SMD:C_1206_3216Metric, symbol Device:C
- added C29, C30, C31, C33, C34: 100nF 10% 50V X7R 0805, Capacitor_SMD:C_0805_2012Metric, symbol Device:C
- added C37, C38: 1uF 10% 100V X7R 1206, Capacitor_SMD:C_1206_3216Metric, symbol Device:C
- added D16, D4: MBRB20200CT, Package_TO_SOT_SMD:TO-263-2, symbol Device:D_Schottky_Dual_CommonCathode_AKA_Parallel
- added D17: SS110, Diode_SMD:D_SMA_Handsoldering, symbol Diode:SS110
- added K1: G5LE-1, Relay_THT:Relay_SPDT_Omron-G5LE-1, symbol Relay:G5LE-1
- added Q1: MMBT3904LT1G, Package_TO_SOT_SMD:SOT-23, symbol Transistor_BJT:MMBT3904
- added Q3: IPP200N25N3, Package_TO_SOT_THT:TO-220-3_Vertical, symbol Transistor_FET:IPP060N06N
- added R1, R3, R38, R39, R5, R55, R56, R57, R58, R8: 10K 1% 0805, Resistor_SMD:R_0805_2012Metric, symbol Device:R_US
- added R29: 100m 3W 1% 2512, Resistor_SMD:R_2512_6332Metric, symbol Device:R_US
- added R31, R37: 4.7K 1% 0805, Resistor_SMD:R_0805_2012Metric, symbol Device:R_US
- added R4: 2.7K 1% 0805, Resistor_SMD:R_0805_2012Metric, symbol Device:R_US
- added R6: 100R 1% 0805, Resistor_SMD:R_0805_2012Metric, symbol Device:R_US
- added U5: OPA171AIDBVR, Package_TO_SOT_SMD:SOT-23-5, symbol Amplifier_Operational:MCP601-xOT
- C14: LCSC Part C5116053 -> (none)
- C15: value 1000uF 100V Electrolytic D18 -> 22uF 100V Electrolytic; footprint Capacitor_THT:CP_Radial_D18.0mm_P7.50mm -> Capacitor_THT:CP_Radial_D6.3mm_P2.50mm; LCSC Part C3445915 -> (none); now left out of the parts list
- C16: value 1nF 1000V -> 1nF 10% 1KV X7R 1206; footprint (none) -> Capacitor_SMD:C_1206_3216Metric; now in the parts list
- C17: LCSC Part C3445915 -> (none); now left out of the parts list
- D1, D5: footprint Diode_SMD:D_SMA -> Diode_SMD:D_SMA_Handsoldering
- D9: value BZX84C15 -> BZX84C15LT1G; LCSC Part (none) -> C80857
- J3, J4: LCSC Part C8446 -> (none)
- L1, L2: value Aprox 220uH -> 1mH 2.4A; footprint Inductor_THT:L_Toroid_Vertical_L25.4mm_W14.7mm_P12.20mm_Vishay_TJ5_BigPads -> Inductor_THT:L_Toroid_Vertical_L31.8mm_W15.9mm_P13.50mm_Bourns_5700
- NT1, NT2: footprint NetTie:NetTie-2_SMD_Pad2.0mm -> NetTie:NetTie-2_SMD_Pad0.5mm
- Q2: now left out of the parts list
- R20: value 33R 1% 0805 Resistor -> 33R 1% 0805; footprint Resistor_SMD:R_0805_2012Metric_Pad1.20x1.40mm_HandSolder -> Resistor_SMD:R_0805_2012Metric; LCSC Part C2907220 -> (none)
- R23: value 10K 1% 0805 Resistor -> 10K 1% 0805; footprint Resistor_SMD:R_0805_2012Metric_Pad1.20x1.40mm_HandSolder -> Resistor_SMD:R_0805_2012Metric; LCSC Part C2907220 -> (none)
- R25: value 10mOhm 3W 1% 2512 -> 10m 3W 1% 2512; footprint Resistor_SMD:R_2512_6332Metric_Pad1.40x3.35mm_HandSolder -> Resistor_SMD:R_2512_6332Metric
- R27: value 4.7R Ohm 3W 1% 2512 -> 4.7R 3W 1% 2512; footprint Resistor_SMD:R_2512_6332Metric_Pad1.40x3.35mm_HandSolder -> Resistor_SMD:R_2512_6332Metric
- U4: value TC4422 -> TC4422ESM
Connections:
- net +12V: now also C33.1, C34.1, C37.1, C38.1, D17.1 (K), K1.2, U5.5 (V+)
- net GNDPWR: now also C34.2, C38.2, D4.1 (A), D4.3 (A), Q1.2 (E), R29.1, R55.1, R56.1, R58.1
- net VIN: now also D4.2 (K)
- net VPWR: now also K1.4; no longer NT2.1, R25.2
- net at C14.2, L2.1: now also C26.2, C32.2, C35.2, C36.2, C39.2, C46.2, D16.1 (A), D16.3 (A)
- net at C14.1, L1.2, Q2.2 (D)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: now also C26.1, C32.1, C35.1, C36.1, C39.1, C46.1
- net Vout renamed VOUT
- net VOUT: now also D16.2 (K)
- new net: Q3.3 (S), R29.2, R8.1
- new net: R38.1, R55.2
- new net: C29.1, R1.2, R3.1
- new net: Q3.1 (G), R6.1
- new net: C31.1, R5.2, R6.2, U5.1
- new net: Q1.1 (B), R31.1, R37.1
- new net: C31.2, R8.2, U5.4 (-)
- new net: C30.1, R3.2, R4.2, U5.3 (+)
- new net: R57.1, R58.2
- new net: R39.1, R56.2
- new net CurveTracer: K1.3, Q3.2 (D)
- new net GNDA: C29.2, C30.2, C33.2, C37.2, R4.1, R5.1, U5.2 (V-)
- new net Tracer_Coil: D17.2 (A), K1.5, Q1.3 (C)
- new net Tracer_En: R31.2, R37.2
- new net Tracer_pwm: R1.1
- new net V_Bleed: K1.1, NT2.1, R25.2, R38.2, R39.2, R57.2
Other:
- moved on the sheet: C14, C15, C16, C17, D1, D5, D9, J13, J14, J3, J4, L1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
