File: hardware/Proyecto0.1V.kicad_sch (KiCad schematic)
At the start: 0 parts

Commit message: Hw/placa sepic (#34)
Co-authored-by: Federico Borello <156438142+fborello-lambda@users.noreply.github.com>
Other:
- sheet Pico ports: added Tracer_En, Tracer_pwm; removed none
- sheet SepicConverter ports: added Tracer_En, Tracer_pwm, VOUT; removed Vout
